Commit message: changed joint names in transmission and bbot_control.yaml file

File: bbot_description/urdf/bbot.transmission.xacro (robot description, xacro)
@@ -5,5 +5,5 @@
       <robotNamespace>/${robot_name}</robotNamespace>
       <type>transmission_interface/SimpleTransmission</type>
-      <joint name="${robot_name}_joint_motor1_link1_2">
+      <joint name="${robot_name}_joint_1">
         <hardwareInterface>hardware_interface/${hardware_interface}</hardwareInterface>
       </joint>
@@ -16,5 +16,5 @@
       <robotNamespace>/${robot_name}</robotNamespace>
       <type>transmission_interface/SimpleTransmission</type>
-      <joint name="${robot_name}_joint_motor2_link2_3">
+      <joint name="${robot_name}_joint_2">
         <hardwareInterface>hardware_interface/${hardware_interface}</hardwareInterface>
       </joint>
@@ -27,5 +27,5 @@
       <robotNamespace>/${robot_name}</robotNamespace>
       <type>transmission_interface/SimpleTransmission</type>
-      <joint name="${robot_name}_joint_link2_3_motor3">
+      <joint name="${robot_name}_joint_3">
         <hardwareInterface>hardware_interface/${hardware_interface}</hardwareInterface>
       </joint>
@@ -38,5 +38,5 @@
       <robotNamespace>/${robot_name}</robotNamespace>
       <type>transmission_interface/SimpleTransmission</type>
-      <joint name="${robot_name}_joint_motor4_link4_5">
+      <joint name="${robot_name}_joint_4">
         <hardwareInterface>hardware_interface/${hardware_interface}</hardwareInterface>
       </joint>
@@ -49,5 +49,5 @@
       <robotNamespace>/${robot_name}</robotNamespace>
       <type>transmission_interface/SimpleTransmission</type>
-      <joint name="${robot_name}_joint_link4_5_motor5">
+      <joint name="${robot_name}_joint_5">
         <hardwareInterface>hardware_interface/${hardware_interface}</hardwareInterface>
       </joint>
@@ -60,5 +60,5 @@
       <robotNamespace>/${robot_name}</robotNamespace>
       <type>transmission_interface/SimpleTransmission</type>
-      <joint name="${robot_name}_joint_link5_6_motor6">
+      <joint name="${robot_name}_joint_6">
         <hardwareInterface>hardware_interface/${hardware_interface}</hardwareInterface>
       </joint>

Commit message: Added transmission and controller config values for bbot_joint_7

File: bbot_description/urdf/bbot.transmission.xacro (robot description, xacro)
@@ -68,4 +68,15 @@
       </actuator>
     </transmission>
+    <transmission name="${robot_name}_tran_7">
+      <robotNamespace>/${robot_name}</robotNamespace>
+      <type>transmission_interface/SimpleTransmission</type>
+      <joint name="${robot_name}_joint_7">
+        <hardwareInterface>hardware_interface/${hardware_interface}</hardwareInterface>
+      </joint>
+      <actuator name="${robot_name}_motor_7">
+        <hardwareInterface>hardware_interface/${hardware_interface}</hardwareInterface>
+        <mechanicalReduction>1</mechanicalReduction>
+      </actuator>
+    </transmission>
   </xacro:macro>
 </robot>
