Commit message: Successfully added aruco ID 99 to gazebo. Still need to exactly position it, and add more markers

File: bbot_description/urdf/ingredient_cup.urdf (robot description, URDF)
Before this commit: robot ingredient_cup, 4 links, 3 joints
Links:
- link aruco_marker: geometry collision mesh filename=package://bbot_aruco/markers/aruco_99_50mm.dae; visual mesh filename=package://bbot_aruco/markers/aruco_99_50mm.dae
Joints:
- joint joint_holder_to_aruco: origin xyz=0 0 0 rpy=0 1.57 0 -> xyz=0 0.03 -0.0025 rpy=0 3.1415 3.1415
