Commit message: Updated mixing cup aruco pose

File: bbot_description/urdf/mixing_cup.xacro (robot description, xacro)
@@ -68,5 +68,5 @@
 	            <parent link="aruco_holder"/>
 	            <child link="aruco_marker"/>
-	            <origin xyz="0 0.0325 0.001" rpy="0 3.1415 3.1415"/>
+	            <origin xyz="0 0.0375 0.001" rpy="0 3.1415 3.1415"/>
 	    </joint>
 		<link name="aruco_marker">
