Commit message: Added stls for links 4_5 and 5_6 and progressed on bbot xacro

File: bbot_description/urdf/bbot.gazebo.xacro (robot description, xacro)
@@ -14,5 +14,5 @@
             <mu2>0.2</mu2>
         </gazebo>
-        <gazebo reference="${robot_name}_link_1_2">
+        <gazebo reference="${robot_name}_link1_2">
             <material>Gazebo/Orange</material>
             <mu1>0.2</mu1>
@@ -24,5 +24,5 @@
             <mu2>0.2</mu2>
         </gazebo>
-        <gazebo reference="${robot_name}_link_2_3">
+        <gazebo reference="${robot_name}_link2_3">
             <material>Gazebo/Orange</material>
             <mu1>0.2</mu1>
@@ -34,5 +34,5 @@
             <mu2>0.2</mu2>
         </gazebo>
-        <gazebo reference="${robot_name}_link_3_4">
+        <gazebo reference="${robot_name}_link3_4">
             <material>Gazebo/Orange</material>
             <mu1>0.2</mu1>
@@ -44,5 +44,5 @@
             <mu2>0.2</mu2>
         </gazebo>
-        <gazebo reference="${robot_name}_link_4_5">
+        <gazebo reference="${robot_name}_link4_5">
             <material>Gazebo/Orange</material>
             <mu1>0.2</mu1>
@@ -54,5 +54,5 @@
             <mu2>0.2</mu2>
         </gazebo>
-        <gazebo reference="${robot_name}_link_5_6">
+        <gazebo reference="${robot_name}_link5_6">
             <material>Gazebo/Orange</material>
             <mu1>0.2</mu1>
@@ -64,5 +64,5 @@
             <mu2>0.2</mu2>
         </gazebo>
-        <gazebo reference="${robot_name}_link_6_7">
+        <gazebo reference="${robot_name}_link6_7">
             <material>Gazebo/Orange</material>
             <mu1>0.2</mu1>

File: bbot_description/urdf/bbot.xacro (robot description, xacro)
@@ -39,8 +39,8 @@
             </collision>
         </link>
-        <joint name="${robot_name}_base_motor1" type="fixed">
+        <joint name="${robot_name}_joint_base_motor1" type="fixed">
             <parent link="${robot_name}_link_baseplate"/>
             <child link="${robot_name}_link_motor1"/>
-            <origin xyz="0 0 0.00719" rpy="0 0 0"/>
+            <origin xyz="0 0 0.01" rpy="0 0 0"/>
         </joint>
         <link name="${robot_name}_link_motor1">
@@ -99,24 +99,24 @@
             </collision>
         </link>
-        <joint name="${robot_name}_link1_2_motor2" type="fixed">
+        <joint name="${robot_name}_joint_link1_2_motor2" type="fixed">
             <parent link="${robot_name}_link1_2"/>
             <child link="${robot_name}_link_motor2"/>
-            <origin xyz="0 0 0.00719" rpy="0 0 0"/>
+            <origin xyz="0 0 0.1" rpy="${pi/2.0} ${-pi/2.0} 0"/>
         </joint>
         <link name="${robot_name}_link_motor2">
             <inertial>
-                <origin xyz="0 0 0.2" rpy="${pi/2} 0 ${pi}"/>
-                <mass value="1"/>
-                <inertia ixx="1.0" ixy="0" ixz="0" iyy="1" iyz="0" izz="1"/>
-            </inertial>
-            <visual>
-                <origin xyz="0 0 0.2" rpy="${pi/2} 0 ${pi}"/>
-                <geometry>
-                    <mesh filename="package://bbot_description/meshes/motor_with_idler.stl" scale="0.001 0.001 0.001"/>
-                </geometry>
-                <material name="Black"/>
-            </visual>
-            <collision>
-                <origin xyz="0 0 0" rpy="${pi/2} 0 ${pi}"/>
+                <origin xyz="0 0 0" rpy="0 0 ${-pi/2.0}"/>
+                <mass value="1"/>
+                <inertia ixx="1.0" ixy="0" ixz="0" iyy="1" iyz="0" izz="1"/>
+            </inertial>
+            <visual>
+                <origin xyz="0 0 0" rpy="0 0 ${-pi/2.0}"/>
+                <geometry>
+                    <mesh filename="package://bbot_description/meshes/motor_with_idler.stl" scale="0.001 0.001 0.001"/>
+                </geometry>
+                <material name="Black"/>
+            </visual>
+            <collision>
+                <origin xyz="0 0 0" rpy="0 0 ${-pi/2.0}"/>
                 <geometry>
                     <mesh filename="package://bbot_description/meshes/motor_with_idler.stl" scale="0.001 0.001 0.001"/>
@@ -140,4 +140,158 @@
         <link name="${robot_name}_link2_3">
             <inertial>
+                <origin xyz="0.1 0 0" rpy="${pi/2.0} ${-pi/2.0} 0"/>
+                <mass value="1"/>
+                <inertia ixx="1.0" ixy="0" ixz="0" iyy="1" iyz="0" izz="1"/>
+            </inertial>
+            <visual>
+                <origin xyz="0.1 0 0" rpy="${pi/2.0} ${-pi/2.0} 0"/>
+                <geometry>
+                    <mesh filename="package://bbot_description/meshes/link2_3.stl" scale="0.001 0.001 0.001"/>
+                </geometry>
+                <material name="Orange"/>
+            </visual>
+            <collision>
+                <origin xyz="0.1 0 0" rpy="${pi/2.0} ${-pi/2.0} 0"/>
+                <geometry>
+                    <mesh filename="package://bbot_description/meshes/link2_3.stl" scale="0.001 0.001 0.001"/>
+                </geometry>
+                <material name="Orange"/>
+            </collision>
+        </link>
+        <joint name="${robot_name}_joint_link2_3_motor3" type="revolute">
+            <parent link="${robot_name}_link2_3"/>
+            <child link="${robot_name}_link_motor3"/>
+            <origin xyz="0.2 0 0" rpy="0 0 0"/>
+            <axis xyz="0 0 1"/>
+            <limit lower="${-170 * pi / 180}" upper="${170 * pi / 180}"
+                effort="${max_effort}" velocity="${max_velocity}" />
+            <safety_controller soft_lower_limit="${-168 * pi / 180}"
+                     soft_upper_limit="${168 * pi / 180}"
+                     k_position="${safety_controller_k_pos}"
+                     k_velocity="${safety_controller_k_vel}"/>
+            <dynamics damping="${joint_damping}"/>
+        </joint>
+        <link name="${robot_name}_link_motor3">
+            <inertial>
+                <origin xyz="0 0 0" rpy="0 0 ${pi/2.0}"/>
+                <mass value="1"/>
+                <inertia ixx="1.0" ixy="0" ixz="0" iyy="1" iyz="0" izz="1"/>
+            </inertial>
+            <visual>
+                <origin xyz="0 0 0" rpy="0 0 ${pi/2.0}"/>
+                <geometry>
+                    <mesh filename="package://bbot_description/meshes/motor_with_idler.stl" scale="0.001 0.001 0.001"/>
+                </geometry>
+                <material name="Black"/>
+            </visual>
+            <collision>
+                <origin xyz="0 0 0" rpy="0 0 ${pi/2.0}"/>
+                <geometry>
+                    <mesh filename="package://bbot_description/meshes/motor_with_idler.stl" scale="0.001 0.001 0.001"/>
+                </geometry>
+                <material name="Black"/>
+            </collision>
+        </link>
+        <joint name="${robot_name}_joint_motor3_link3_4" type="fixed">
+            <parent link="${robot_name}_link_motor3"/>
+            <child link="${robot_name}_link3_4"/>
+            <origin xyz="0 0 0" rpy="0 0 0"/>
+        </joint>
+        <link name="${robot_name}_link3_4">
+            <inertial>
+                <origin xyz="0.1 0 0" rpy="0 0 0"/>
+                <mass value="1"/>
+                <inertia ixx="1.0" ixy="0" ixz="0" iyy="1" iyz="0" izz="1"/>
+            </inertial>
+            <visual>
+                <origin xyz="0.1 0 0" rpy="0 0 0"/>
+                <geometry>
+                    <mesh filename="package://bbot_description/meshes/link3_4.stl" scale="0.001 0.001 0.001"/>
+                </geometry>
+                <material name="Orange"/>
+            </visual>
+            <collision>
+                <origin xyz="0.1 0 0" rpy="0 0 0"/>
+                <geometry>
+                    <mesh filename="package://bbot_description/meshes/link3_4.stl" scale="0.001 0.001 0.001"/>
+                </geometry>
+                <material name="Orange"/>
+            </collision>
+        </link>
+        <joint name="${robot_name}_joint_link3_4_motor4" type="fixed">
+            <parent link="${robot_name}_link3_4"/>
+            <child link="${robot_name}_link_motor4"/>
+            <origin xyz="0.2 0 0" rpy="0 0 0"/>
+        </joint>
+        <link name="${robot_name}_link_motor4">
+            <inertial>
+                <origin xyz="0 0 0" rpy="0 0 ${pi/2.0}"/>
+                <mass value="1"/>
+                <inertia ixx="1.0" ixy="0" ixz="0" iyy="1" iyz="0" izz="1"/>
+            </inertial>
+            <visual>
+                <origin xyz="0 0 0" rpy="0 0 ${pi/2.0}"/>
+                <geometry>
+                    <mesh filename="package://bbot_description/meshes/motor_with_idler.stl" scale="0.001 0.001 0.001"/>
+                </geometry>
+                <material name="Black"/>
+            </visual>
+            <collision>
+                <origin xyz="0 0 0" rpy="0 0 ${pi/2.0}"/>
+                <geometry>
+                    <mesh filename="package://bbot_description/meshes/motor_with_idler.stl" scale="0.001 0.001 0.001"/>
+                </geometry>
+                <material name="Black"/>
+            </collision>
+        </link>
+        <joint name="${robot_name}_joint_motor4_link4_5" type="revolute">
+            <parent link="${robot_name}_link_motor4"/>
+            <child link="${robot_name}_link4_5"/>
+            <origin xyz="0 0 0" rpy="0 0 0"/>
+            <axis xyz="0 0 1"/>
+            <limit lower="${-170 * pi / 180}" upper="${170 * pi / 180}"
+                effort="${max_effort}" velocity="${max_velocity}" />
+            <safety_controller soft_lower_limit="${-168 * pi / 180}"
+                     soft_upper_limit="${168 * pi / 180}"
+                     k_position="${safety_controller_k_pos}"
+                     k_velocity="${safety_controller_k_vel}"/>
+            <dynamics damping="${joint_damping}"/>
+        </joint>
+        <link name="${robot_name}_link4_5">
+            <inertial>
+                <origin xyz="0 0 0.1" rpy="0 0 0"/>
+                <mass value="1"/>
+                <inertia ixx="1.0" ixy="0" ixz="0" iyy="1" iyz="0" izz="1"/>
+            </inertial>
+            <visual>
+                <origin xyz="0 0 0.1" rpy="0 0 0"/>
+                <geometry>
+                    <mesh filename="package://bbot_description/meshes/link4_5.stl" scale="0.001 0.001 0.001"/>
+                </geometry>
+                <material name="Orange"/>
+            </visual>
+            <collision>
+                <origin xyz="0 0 0.1" rpy="0 0 0"/>
+                <geometry>
+                    <mesh filename="package://bbot_description/meshes/link4_5.stl" scale="0.001 0.001 0.001"/>
+                </geometry>
+                <material name="Orange"/>
+            </collision>
+        </link>
+        <joint name="${robot_name}_joint_link4_5_motor5" type="revolute">
+            <parent link="${robot_name}_link4_5"/>
+            <child link="${robot_name}_link_motor5"/>
+            <origin xyz="0 0 0.15" rpy="${pi/2.0} ${-pi/2.0} 0"/>
+            <axis xyz="0 0 1"/>
+            <limit lower="${-170 * pi / 180}" upper="${170 * pi / 180}"
+                effort="${max_effort}" velocity="${max_velocity}" />
+            <safety_controller soft_lower_limit="${-168 * pi / 180}"
+                     soft_upper_limit="${168 * pi / 180}"
+                     k_position="${safety_controller_k_pos}"
+                     k_velocity="${safety_controller_k_vel}"/>
+            <dynamics damping="${joint_damping}"/>
+        </joint>
+        <link name="${robot_name}_link_motor5">
+            <inertial>
                 <origin xyz="0 0 0" rpy="0 0 0"/>
                 <mass value="1"/>
@@ -147,28 +301,76 @@
                 <origin xyz="0 0 0" rpy="0 0 0"/>
                 <geometry>
-                    <mesh filename="package://bbot_description/meshes/link2_3.stl" scale="0.001 0.001 0.001"/>
-                </geometry>
-                <material name="Orange"/>
+                    <mesh filename="package://bbot_description/meshes/motor_with_idler.stl" scale="0.001 0.001 0.001"/>
+                </geometry>
+                <material name="Black"/>
             </visual>
             <collision>
                 <origin xyz="0 0 0" rpy="0 0 0"/>
                 <geometry>
-                    <mesh filename="package://bbot_description/meshes/link2_3.stl" scale="0.001 0.001 0.001"/>
-                </geometry>
-                <material name="Orange"/>
-            </collision>
-        </link>
-        <!-- joint between motor 2 and link2_3 -->
-        <!-- link 2_3 -->
-        <!-- joint between link2_3 and motor 3 -->
-        <!-- motor3 as link-->
-        <!-- joint between motor 3 and link 3_4 -->
-        <!-- link 3_4 -->
-        <!-- joint between link 3_4 and motor 4 -->
-        <!-- motor4 -->
-        <!-- joint between motor 4 and link 4_5 -->
-        <!-- link 4_5 -->
-        <!-- joint between link 4_5 and motor 5 -->
-        <!-- motor 5 -->
+                    <mesh filename="package://bbot_description/meshes/motor_with_idler.stl" scale="0.001 0.001 0.001"/>
+                </geometry>
+                <material name="Black"/>
+            </collision>
+        </link>
+        <joint name="${robot_name}_joint_motor5_link5_6" type="fixed">
+            <parent link="${robot_name}_link_motor5"/>
+            <child link="${robot_name}_link5_6"/>
+            <origin xyz="0 -0.1 0" rpy="0 0 0"/>
+        </joint>
+        <link name="${robot_name}_link5_6">
+            <inertial>
+                <origin xyz="0 0 0" rpy="${pi/2.0} 0 ${pi/2.0}"/>
+                <mass value="1"/>
+                <inertia ixx="1.0" ixy="0" ixz="0" iyy="1" iyz="0" izz="1"/>
+            </inertial>
+            <visual>
+                <origin xyz="0 0 0" rpy="${pi/2.0} 0 ${pi/2.0}"/>
+                <geometry>
+                    <mesh filename="package://bbot_description/meshes/link5_6.stl" scale="0.001 0.001 0.001"/>
+                </geometry>
+                <material name="Orange"/>
+            </visual>
+            <collision>
+                <origin xyz="0 0 0" rpy="${pi/2.0} 0 ${pi/2.0}"/>
+                <geometry>
+                    <mesh filename="package://bbot_description/meshes/link5_6.stl" scale="0.001 0.001 0.001"/>
+                </geometry>
+                <material name="Orange"/>
+            </collision>
+        </link>
+        <joint name="${robot_name}_joint_link5_6_motor6" type="revolute">
+            <parent link="${robot_name}_link5_6"/>
+            <child link="${robot_name}_link_motor6"/>
+            <origin xyz="0 -0.1 0" rpy="${pi/2.0} 0 0"/>
+            <axis xyz="0 0 1"/>
+            <limit lower="${-170 * pi / 180}" upper="${170 * pi / 180}"
+                effort="${max_effort}" velocity="${max_velocity}" />
+            <safety_controller soft_lower_limit="${-168 * pi / 180}"
+                     soft_upper_limit="${168 * pi / 180}"
+                     k_position="${safety_controller_k_pos}"
+                     k_velocity="${safety_controller_k_vel}"/>
+            <dynamics damping="${joint_damping}"/>
+        </joint>
+        <link name="${robot_name}_link_motor6">
+            <inertial>
+                <origin xyz="0 0 0" rpy="0 0 ${pi}"/>
+                <mass value="1"/>
+                <inertia ixx="1.0" ixy="0" ixz="0" iyy="1" iyz="0" izz="1"/>
+            </inertial>
+            <visual>
+                <origin xyz="0 0 0" rpy="0 0 ${pi}"/>
+                <geometry>
+                    <mesh filename="package://bbot_description/meshes/motor_with_idler.stl" scale="0.001 0.001 0.001"/>
+                </geometry>
+                <material name="Black"/>
+            </visual>
+            <collision>
+                <origin xyz="0 0 0" rpy="0 0 ${pi}"/>
+                <geometry>
+                    <mesh filename="package://bbot_description/meshes/motor_with_idler.stl" scale="0.001 0.001 0.001"/>
+                </geometry>
+                <material name="Black"/>
+            </collision>
+        </link>
         <!-- joint between motor 5 and link 5_6 -->
         <!-- link 5_6 -->

Commit message: Got the gazebo bbot controlled using position controllers

File: bbot_description/urdf/bbot.gazebo.xacro (robot description, xacro)
@@ -2,4 +2,10 @@
 <robot xmlns:xacro="http://www.ros.org/wiki/xacro">
     <xacro:macro name="bbot_gazebo" params="robot_name">
+        <!-- Load Gazebo lib and set the robot namespace -->
+        <gazebo>
+            <plugin name="gazebo_ros_control" filename="libgazebo_ros_control.so">
+                <robotNamespace>/${robot_name}</robotNamespace>
+            </plugin>
+        </gazebo>
         <!-- Link0 -->
         <gazebo reference="${robot_name}_link_baseplate">

File: bbot_description/urdf/bbot.urdf.xacro (robot description, xacro)
@@ -5,12 +5,14 @@
 	<!-- Import the bbot macro -->
 	<xacro:include filename="$(find bbot_description)/urdf/bbot.xacro"/>
+  <!-- arguments to pass on -->
+  <xacro:arg name="hardware_interface" default="PositionJointInterface"/>
 	<xacro:arg name="robot_name" default="bbot"/>
 	<xacro:arg name="origin_xyz" default="0 0 0"/>
-  	<xacro:arg name="origin_rpy" default="0 0 0"/>
-  	<!-- Fix to world-->
-  	<link name="world"/>
-  	<!-- call bbot xacro -->
-  	<xacro:bbot robot_name="$(arg robot_name)" parent="world">
-  		<origin xyz="$(arg origin_xyz)" rpy="$(arg origin_rpy)"/>
-  	</xacro:bbot>
+  <xacro:arg name="origin_rpy" default="0 0 0"/>
+  <!-- Fix to world-->
+  <link name="world"/>
+  <!-- call bbot xacro -->
+  <xacro:bbot hardware_interface="$(arg hardware_interface)" robot_name="$(arg robot_name)" parent="world">
+  	<origin xyz="$(arg origin_xyz)" rpy="$(arg origin_rpy)"/>
+  </xacro:bbot>
 </robot>

File: bbot_description/urdf/bbot.xacro (robot description, xacro)
@@ -3,5 +3,6 @@
     <!-- Import all Gazebo customization elements including colors-->
     <xacro:include filename="$(find bbot_description)/urdf/bbot.gazebo.xacro"/>
-    <!-- Import transmissions -->
+    <!-- Import Transmissions -->
+    <xacro:include filename="$(find bbot_description)/urdf/bbot.transmission.xacro" />
     <!-- Include Utilities -->
     <!--Define properties-->
@@ -11,5 +12,5 @@
     <xacro:property name="max_effort" value="300"/>
     <xacro:property name="max_velocity" value="10"/>
-    <xacro:macro name="bbot" params="parent robot_name *origin">
+    <xacro:macro name="bbot" params="parent hardware_interface robot_name *origin">
         <!-- joint between parent (a.k.a. world) and link_0 -->
         <joint name="${parent}_${robot_name}_joint" type="fixed">
@@ -384,4 +385,5 @@
         <!-- link_claw1 -->
         <xacro:bbot_gazebo robot_name="${robot_name}"/>
+        <xacro:bbot_transmission hardware_interface="${hardware_interface}"/>
     </xacro:macro>
 </robot>

Commit message: Rename Joint 7

File: bbot_description/urdf/bbot.gazebo.xacro (robot description, xacro)
@@ -80,4 +80,34 @@
             <mu2>0.2</mu2>
         </gazebo>
+        <gazebo reference="${robot_name}_link_claw1">
+            <material>Gazebo/Orange</material>
+            <mu1>0.2</mu1>
+            <mu2>0.2</mu2>
+        </gazebo>
+        <gazebo reference="${robot_name}_link_claw1_end">
+            <material>Gazebo/Orange</material>
+            <mu1>0.2</mu1>
+            <mu2>0.2</mu2>
+        </gazebo>
+        <gazebo reference="${robot_name}_link_claw1_2">
+            <material>Gazebo/Orange</material>
+            <mu1>0.2</mu1>
+            <mu2>0.2</mu2>
+        </gazebo>
+        <gazebo reference="${robot_name}_link_claw2">
+            <material>Gazebo/Orange</material>
+            <mu1>0.2</mu1>
+            <mu2>0.2</mu2>
+        </gazebo>
+        <gazebo reference="${robot_name}_link_claw2_end">
+            <material>Gazebo/Orange</material>
+            <mu1>0.2</mu1>
+            <mu2>0.2</mu2>
+        </gazebo>
+        <gazebo reference="${robot_name}_link_claw2_2">
+            <material>Gazebo/Orange</material>
+            <mu1>0.2</mu1>
+            <mu2>0.2</mu2>
+        </gazebo>
     </xacro:macro>
 </robot>

File: bbot_description/urdf/bbot.xacro (robot description, xacro)
@@ -431,5 +431,5 @@
         </link>
         <!-- joint between motor 7 and link_claw1-->
-        <joint name="${robot_name}_joint_motor7_claw1" type="revolute">
+        <joint name="${robot_name}_joint_7" type="revolute">
             <parent link="${robot_name}_link_motor7"/>
             <child link="${robot_name}_link_claw1"/>
@@ -528,5 +528,5 @@
             <origin xyz="0.03 0 0" rpy="0 0 0"/>
         </joint> -->
-        <!-- link_claw2_2 -->
+        <!-- link_claw2 -->
 <!--         <link name="${robot_name}_link_claw2">
             <inertial>
