Commit message: Uncommented rest of BBOT

File: bbot_description/urdf/bbot.gazebo.xacro (robot description, xacro)
@@ -75,4 +75,9 @@
             <mu2>0.2</mu2>
         </gazebo>
+        <gazebo reference="${robot_name}_gripper_palm">
+            <material>Gazebo/Orange</material>
+            <mu1>0.2</mu1>
+            <mu2>0.2</mu2>
+        </gazebo>
         <gazebo reference="${robot_name}_link_motor7">
             <material>Gazebo/Black</material>

File: bbot_description/urdf/bbot.xacro (robot description, xacro)
@@ -467,11 +467,11 @@
         </link>
         <!-- joint between link_claw1 and link_claw1_end-->
-<!--         <joint name="${robot_name}_joint_claw1_claw1_end" type="fixed">
+        <joint name="${robot_name}_joint_claw1_claw1_end" type="fixed">
             <parent link="${robot_name}_link_claw1"/>
             <child link="${robot_name}_link_claw1_end"/>
             <origin xyz="-0.03677 -0.03677 -0.00825" rpy="0 0 0"/>
-        </joint> -->
+        </joint>
         <!-- link_claw1_end -->
-<!--         <link name="${robot_name}_link_claw1_end">
+        <link name="${robot_name}_link_claw1_end">
             <inertial>
                 <origin xyz="0.01175 -0.0276 0.00325" rpy="${pi/2} 0 1.903"/>
@@ -493,13 +493,13 @@
                 <material name="Orange"/>
             </collision>
-        </link> -->
+        </link>
         <!-- joint between link_claw1_end and link_claw1_2-->
-<!--         <joint name="${robot_name}_joint_claw1_end_claw1_2" type="fixed">
+        <joint name="${robot_name}_joint_claw1_end_claw1_2" type="fixed">
             <parent link="${robot_name}_link_claw1_end"/>
             <child link="${robot_name}_link_claw1_2"/>
             <origin xyz="0.0098 -0.023 0.00025" rpy="0 0 0"/>
-        </joint> -->
+        </joint>
         <!-- link_claw1_2 -->
-<!--         <link name="${robot_name}_link_claw1_2">
+        <link name="${robot_name}_link_claw1_2">
             <inertial>
                 <origin xyz="0.01839 0.01693 0.0135" rpy="${-pi/2} 0 -2.3057"/>
@@ -521,13 +521,13 @@
                 <material name="Orange"/>
             </collision>
-        </link> -->
+        </link>
         <!-- joint between link_claw1 and link_claw2-->
-<!--         <joint name="${robot_name}_joint_claw1_claw2" type="fixed">
+        <joint name="${robot_name}_joint_claw1_claw2" type="fixed">
             <parent link="${robot_name}_link_claw1"/>
             <child link="${robot_name}_link_claw2"/>
             <origin xyz="0.03 0 0" rpy="0 0 0"/>
-        </joint> -->
+        </joint>
         <!-- link_claw2 -->
-<!--         <link name="${robot_name}_link_claw2">
+        <link name="${robot_name}_link_claw2">
             <inertial>
                 <origin xyz="0 0 0.005" rpy="0 ${pi} ${pi}"/>
@@ -550,13 +550,12 @@
             </collision>
         </link>
- -->
         <!-- joint between link_claw2 and link_claw2_end-->
-<!--         <joint name="${robot_name}_joint_claw2_claw2_end" type="fixed">
+        <joint name="${robot_name}_joint_claw2_claw2_end" type="fixed">
             <parent link="${robot_name}_link_claw2"/>
             <child link="${robot_name}_link_claw2_end"/>
             <origin xyz="0.03581 -0.0377 -0.0085" rpy="0 0 0"/>
-        </joint> -->
+        </joint>
         <!-- link_claw2_end -->
-<!--         <link name="${robot_name}_link_claw2_end">
+        <link name="${robot_name}_link_claw2_end">
             <inertial>
                 <origin xyz="-0.01181 -0.02758 0.0085" rpy="${pi/2} ${pi} -1.903"/>
@@ -578,13 +577,13 @@
                 <material name="Orange"/>
             </collision>
-        </link> -->
+        </link>
         <!-- joint between link_claw2_end and link_claw2_2-->
-<!--         <joint name="${robot_name}_joint_claw1_end_claw2_2" type="fixed">
+        <joint name="${robot_name}_joint_claw1_end_claw2_2" type="fixed">
             <parent link="${robot_name}_link_claw2_end"/>
             <child link="${robot_name}_link_claw2_2"/>
             <origin xyz="-0.00984 -0.02298 0" rpy="0 0 0"/>
-        </joint> -->
+        </joint>
         <!-- link_claw2_2 -->
-<!--         <link name="${robot_name}_link_claw2_2">
+        <link name="${robot_name}_link_claw2_2">
             <inertial>
                 <origin xyz="-0.01699 0.01834 0.0135" rpy="${pi/2} ${pi} 2.3057"/>
@@ -606,5 +605,5 @@
                 <material name="Orange"/>
             </collision>
-        </link> -->
+        </link>
         <xacro:bbot_gazebo robot_name="${robot_name}"/>
         <xacro:bbot_transmission hardware_interface="${hardware_interface}"/>

Commit message: Added mimic plug-in

File: bbot_description/urdf/bbot.gazebo.xacro (robot description, xacro)
@@ -116,3 +116,22 @@
         </gazebo>
     </xacro:macro>
+    <!-- Load in mimic_joint_plugin -->
+    <xacro:macro name="mimic_joint_plugin_gazebo" params="name_prefix parent_joint mimic_joint has_pid:=false multiplier:=1.0 offset:=0 sensitiveness:=0.0 max_effort:=1.0 robot_namespace:=''">
+    <gazebo>
+      <plugin name="${name_prefix}mimic_joint_plugin" filename="libroboticsgroup_gazebo_mimic_joint_plugin.so">
+        <joint>${parent_joint}</joint>
+        <mimicJoint>${mimic_joint}</mimicJoint>
+        <xacro:if value="${has_pid}">                     <!-- if set to true, PID parameters from "/gazebo_ros_control/pid_gains/${mimic_joint}" are loaded -->
+          <hasPID />
+        </xacro:if>
+        <multiplier>${multiplier}</multiplier>
+        <offset>${offset}</offset>
+        <sensitiveness>${sensitiveness}</sensitiveness>   <!-- if absolute difference between setpoint and process value is below this threshold, do nothing; 0.0 = disable [rad] -->
+        <maxEffort>${max_effort}</maxEffort>              <!-- only taken into account if has_pid:=true [Nm] -->
+        <xacro:unless value="${robot_namespace == ''}">
+          <robotNamespace>${robot_namespace}</robotNamespace>
+        </xacro:unless>
+      </plugin>
+    </gazebo>
+  </xacro:macro>
 </robot>

File: bbot_description/urdf/bbot.xacro (robot description, xacro)
@@ -523,9 +523,22 @@
         </link>
         <!-- joint between link_claw1 and link_claw2-->
-        <joint name="${robot_name}_joint_claw1_claw2" type="fixed">
+        <joint name="${robot_name}_joint_claw1_claw2" type="revolute">
             <parent link="${robot_name}_link_claw1"/>
             <child link="${robot_name}_link_claw2"/>
             <origin xyz="0.03 0 0" rpy="0 0 0"/>
-        </joint>
+            <axis xyz="0 0 1"/>
+            <limit lower="${-170 * pi / 180}" upper="${170 * pi / 180}"
+                effort="${max_effort}" velocity="${max_velocity}" />
+            <safety_controller soft_lower_limit="${-168 * pi / 180}"
+                     soft_upper_limit="${168 * pi / 180}"
+                     k_position="${safety_controller_k_pos}"
+                     k_velocity="${safety_controller_k_vel}"/>
+            <dynamics damping="${joint_damping}"/>
+            <mimic joint="${robot_name}_joint_7" multiplier="-1.0" offset = "0.0"/>
+        </joint>
+        <xacro:mimic_joint_plugin_gazebo name_prefix="${robot_name}_joint_claw1_claw2"
+            parent_joint="${robot_name}_joint_7"
+            mimic_joint="${robot_name}_joint_claw1_claw2"
+            has_pid="true" multiplier="-1.0" max_effort="${max_effort}" />
         <!-- link_claw2 -->
         <link name="${robot_name}_link_claw2">

Commit message: Mimic joints working, continuous joints added

File: bbot_description/urdf/bbot.gazebo.xacro (robot description, xacro)
@@ -8,4 +8,14 @@
             </plugin>
         </gazebo>
+        <!-- Load Closed Loop Plug-in -->
+<!--         <gazebo>
+       <plugin name="Myrobot_ClosedLoopPlugin" filename="libpegasus_gazebo_closed_loop_plugin.so">
+           <joint>${robot_name}_joint_claw1_claw1_end_2</joint>
+           <child>${robot_name}_link_claw1_end</child>
+           <parent>${robot_name}_link_claw1_2</parent>
+           <position>-0.03678 -0.03387 0</position>
+           <rotation>0.00 0.00 0.00</rotation>
+       </plugin>
+        </gazebo> -->
         <!-- Link0 -->
         <gazebo reference="${robot_name}_link_baseplate">

File: bbot_description/urdf/bbot.xacro (robot description, xacro)
@@ -466,47 +466,32 @@
             </collision>
         </link>
-        <!-- joint between link_claw1 and link_claw1_end-->
-        <joint name="${robot_name}_joint_claw1_claw1_end" type="fixed">
+        <!-- joint between link_claw1 and link_claw1_2-->
+        <joint name="${robot_name}_joint_claw1_claw1_2" type="revolute">
             <parent link="${robot_name}_link_claw1"/>
-            <child link="${robot_name}_link_claw1_end"/>
-            <origin xyz="-0.03677 -0.03677 -0.00825" rpy="0 0 0"/>
-        </joint>
-        <!-- link_claw1_end -->
-        <link name="${robot_name}_link_claw1_end">
-            <inertial>
-                <origin xyz="0.01175 -0.0276 0.00325" rpy="${pi/2} 0 1.903"/>
-                <mass value="0.006"/>
-                <inertia ixx="0" ixy="0" ixz="0" iyy="0.000003" iyz="0" izz="0.000003"/>
-            </inertial>
-            <visual>
-                <origin xyz="0.01175 -0.0276 0.00325" rpy="${pi/2} 0 1.903"/>
-                <geometry>
-                    <mesh filename="package://bbot_description/meshes/gripper_link3.stl" scale="0.001 0.001 0.001"/>
-                </geometry>
-                <material name="Orange"/>
-            </visual>
-            <collision>
-                <origin xyz="0.01175 -0.0276 0.00325" rpy="${pi/2} 0 1.903"/>
-                <geometry>
-                    <mesh filename="package://bbot_description/meshes/gripper_link3.stl" scale="0.001 0.001 0.001"/>
-                </geometry>
-                <material name="Orange"/>
-            </collision>
-        </link>
-        <!-- joint between link_claw1_end and link_claw1_2-->
-        <joint name="${robot_name}_joint_claw1_end_claw1_2" type="fixed">
-            <parent link="${robot_name}_link_claw1_end"/>
             <child link="${robot_name}_link_claw1_2"/>
-            <origin xyz="0.0098 -0.023 0.00025" rpy="0 0 0"/>
-        </joint>
+            <origin xyz="0.008 -0.024 0" rpy="0 0 0"/>
+            <axis xyz="0 0 1"/>
+            <limit lower="${-170 * pi / 180}" upper="${170 * pi / 180}"
+                effort="${max_effort}" velocity="${max_velocity}" />
+            <safety_controller soft_lower_limit="${-168 * pi / 180}"
+                     soft_upper_limit="${168 * pi / 180}"
+                     k_position="${safety_controller_k_pos}"
+                     k_velocity="${safety_controller_k_vel}"/>
+            <dynamics damping="${joint_damping}"/>
+            <mimic joint="${robot_name}_joint_7" multiplier="1.0" offset = "0.0"/>
+        </joint>
+        <xacro:mimic_joint_plugin_gazebo name_prefix="${robot_name}_joint_claw1_claw1_2"
+            parent_joint="${robot_name}_joint_7"
+            mimic_joint="${robot_name}_joint_claw1_claw1_2"
+            has_pid="false" multiplier="1.0" max_effort="${max_effort}" />
         <!-- link_claw1_2 -->
         <link name="${robot_name}_link_claw1_2">
             <inertial>
-                <origin xyz="0.01839 0.01693 0.0135" rpy="${-pi/2} 0 -2.3057"/>
+                <origin xyz="-0.01839 -0.01693 0.005" rpy="${-pi/2} 0 -2.3057"/>
                 <mass value=".00455"/>
                 <inertia ixx="0" ixy="0" ixz="0" iyy="0.000001" iyz="0" izz="0.000001"/>
             </inertial>
             <visual>
-                <origin xyz="0.01839 0.01693 0.0135" rpy="${-pi/2} 0 -2.3057"/>
+                <origin xyz="-0.01839 -0.01693 0.005" rpy="${-pi/2} 0 -2.3057"/>
                 <geometry>
                     <mesh filename="package://bbot_description/meshes/gripper_link2.stl" scale="0.001 0.001 0.001"/>
@@ -515,5 +500,5 @@
             </visual>
             <collision>
-                <origin xyz="0.01839 0.01693 0.0135" rpy="${-pi/2} 0 -2.3057"/>
+                <origin xyz="-0.01839 -0.01693 0.005" rpy="${-pi/2} 0 -2.3057"/>
                 <geometry>
                     <mesh filename="package://bbot_description/meshes/gripper_link2.stl" scale="0.001 0.001 0.001"/>
@@ -540,14 +525,49 @@
             parent_joint="${robot_name}_joint_7"
             mimic_joint="${robot_name}_joint_claw1_claw2"
-            has_pid="true" multiplier="-1.0" max_effort="${max_effort}" />
+            has_pid="false" multiplier="-1.0" max_effort="${max_effort}" />
+        <!-- joint between link_claw1 and link_claw1_end-->
+        <joint name="${robot_name}_joint_claw1_claw1_end" type="continuous">
+            <parent link="${robot_name}_link_claw1"/>
+            <child link="${robot_name}_link_claw1_end"/>
+            <origin xyz="-0.03858 -0.03487 0" rpy="0 0 0"/>
+            <axis xyz="0 0 1"/>
+        </joint>
+        <!-- link_claw1_end -->
+        <link name="${robot_name}_link_claw1_end">
+            <inertial>
+                <origin xyz="0.01175 -0.0276 -0.005" rpy="${pi/2} 0 1.903"/>
+                <mass value="0.006"/>
+                <inertia ixx="0" ixy="0" ixz="0" iyy="0.000003" iyz="0" izz="0.000003"/>
+            </inertial>
+            <visual>
+                <origin xyz="0.01175 -0.0276 -0.005" rpy="${pi/2} 0 1.903"/>
+                <geometry>
+                    <mesh filename="package://bbot_description/meshes/gripper_link3.stl" scale="0.001 0.001 0.001"/>
+                </geometry>
+                <material name="Orange"/>
+            </visual>
+            <collision>
+                <origin xyz="0.01175 -0.0276 -0.005" rpy="${pi/2} 0 1.903"/>
+                <geometry>
+                    <mesh filename="package://bbot_description/meshes/gripper_link3.stl" scale="0.001 0.001 0.001"/>
+                </geometry>
+                <material name="Orange"/>
+            </collision>
+        </link>
+<!--         <joint name="${robot_name}_joint_claw1_claw1_end_2" type="continuous">
+            <parent link="${robot_name}_link_claw1_2"/>
+            <child link="${robot_name}_link_claw1_end"/>
+            <origin xyz="-0.03678 -0.03387 0" rpy="0 0 0"/>
+            <axis xyz="0 0 1"/>
+        </joint> -->
         <!-- link_claw2 -->
         <link name="${robot_name}_link_claw2">
             <inertial>
-                <origin xyz="0 0 0.005" rpy="0 ${pi} ${pi}"/>
+                <origin xyz="0 0 0.005" rpy="0 ${pi} 3.307"/>
                 <mass value=".0066"/>
                 <inertia ixx="0.000004" ixy="0.000003" ixz="0" iyy="0.000002" iyz="0.000001" izz="0.000006"/>
             </inertial>
             <visual>
-                <origin xyz="0 0 0.005" rpy="0 ${pi} ${pi}"/>
+                <origin xyz="0 0 0.005" rpy="0 ${pi} 3.307"/>
                 <geometry>
                     <mesh filename="package://bbot_description/meshes/gripper_link1_left.stl" scale="0.001 0.001 0.001"/>
@@ -556,5 +576,5 @@
             </visual>
             <collision>
-                <origin xyz="0 0 0.005" rpy="0 ${pi} ${pi}"/>
+                <origin xyz="0 0 0.005" rpy="0 ${pi} 3.307"/>
                 <geometry>
                     <mesh filename="package://bbot_description/meshes/gripper_link1_left.stl" scale="0.001 0.001 0.001"/>
@@ -563,19 +583,61 @@
             </collision>
         </link>
+        <!-- joint between link_claw2 and link_claw2_2-->
+        <joint name="${robot_name}_joint_claw2_claw2_2" type="revolute">
+            <parent link="${robot_name}_link_claw2"/>
+            <child link="${robot_name}_link_claw2_2"/>
+            <origin xyz="-0.008 -0.024 0" rpy="0 0 0"/>
+            <axis xyz="0 0 1"/>
+            <limit lower="${-170 * pi / 180}" upper="${170 * pi / 180}"
+                effort="${max_effort}" velocity="${max_velocity}" />
+            <safety_controller soft_lower_limit="${-168 * pi / 180}"
+                     soft_upper_limit="${168 * pi / 180}"
+                     k_position="${safety_controller_k_pos}"
+                     k_velocity="${safety_controller_k_vel}"/>
+            <dynamics damping="${joint_damping}"/>
+            <mimic joint="${robot_name}_joint_7" multiplier="-1.0" offset = "0.0"/>
+        </joint>
+        <xacro:mimic_joint_plugin_gazebo name_prefix="${robot_name}_joint_claw2_claw2_2"
+            parent_joint="${robot_name}_joint_7"
+            mimic_joint="${robot_name}_joint_claw2_claw2_2"
+            has_pid="false" multiplier="-1.0" max_effort="${max_effort}" />
+        <!-- link_claw2_2 -->
+        <link name="${robot_name}_link_claw2_2">
+            <inertial>
+                <origin xyz="0.01699 -0.01834 0.005" rpy="${pi/2} ${pi} 2.3057"/>
+                <mass value=".00455"/>
+                <inertia ixx="0" ixy="0" ixz="0" iyy="0.000001" iyz="0" izz="0.000001"/>
+            </inertial>
+            <visual>
+                <origin xyz="0.01699 -0.01834 0.005" rpy="${pi/2} ${pi} 2.3057"/>
+                <geometry>
+                    <mesh filename="package://bbot_description/meshes/gripper_link2.stl" scale="0.001 0.001 0.001"/>
+                </geometry>
+                <material name="Orange"/>
+            </visual>
+            <collision>
+                <origin xyz="0.01699 -0.01834 0.005" rpy="${pi/2} ${pi} 2.3057"/>
+                <geometry>
+                    <mesh filename="package://bbot_description/meshes/gripper_link2.stl" scale="0.001 0.001 0.001"/>
+                </geometry>
+                <material name="Orange"/>
+            </collision>
+        </link>
         <!-- joint between link_claw2 and link_claw2_end-->
-        <joint name="${robot_name}_joint_claw2_claw2_end" type="fixed">
+        <joint name="${robot_name}_joint_claw2_claw2_end" type="continuous">
             <parent link="${robot_name}_link_claw2"/>
             <child link="${robot_name}_link_claw2_end"/>
-            <origin xyz="0.03581 -0.0377 -0.0085" rpy="0 0 0"/>
+            <origin xyz="0.03581 -0.0377 0" rpy="0 0 0"/>
+            <axis xyz="0 0 1"/>
         </joint>
         <!-- link_claw2_end -->
         <link name="${robot_name}_link_claw2_end">
             <inertial>
-                <origin xyz="-0.01181 -0.02758 0.0085" rpy="${pi/2} ${pi} -1.903"/>
+                <origin xyz="-0.01181 -0.02758 0" rpy="${pi/2} ${pi} -1.903"/>
                 <mass value="0.006"/>
                 <inertia ixx="0" ixy="0" ixz="0" iyy="0.000003" iyz="0" izz="0.000003"/>
             </inertial>
             <visual>
-                <origin xyz="-0.01181 -0.02758 0.0085" rpy="${pi/2} ${pi} -1.903"/>
+                <origin xyz="-0.01181 -0.02758 0" rpy="${pi/2} ${pi} -1.903"/>
                 <geometry>
                     <mesh filename="package://bbot_description/meshes/gripper_link3.stl" scale="0.001 0.001 0.001"/>
@@ -584,35 +646,7 @@
             </visual>
             <collision>
-                <origin xyz="-0.01181 -0.02758 0.0085" rpy="${pi/2} ${pi} -1.903"/>
+                <origin xyz="-0.01181 -0.02758 0" rpy="${pi/2} ${pi} -1.903"/>
                 <geometry>
                     <mesh filename="package://bbot_description/meshes/gripper_link3.stl" scale="0.001 0.001 0.001"/>
-                </geometry>
-                <material name="Orange"/>
-            </collision>
-        </link>
-        <!-- joint between link_claw2_end and link_claw2_2-->
-        <joint name="${robot_name}_joint_claw1_end_claw2_2" type="fixed">
-            <parent link="${robot_name}_link_claw2_end"/>
-            <child link="${robot_name}_link_claw2_2"/>
-            <origin xyz="-0.00984 -0.02298 0" rpy="0 0 0"/>
-        </joint>
-        <!-- link_claw2_2 -->
-        <link name="${robot_name}_link_claw2_2">
-            <inertial>
-                <origin xyz="-0.01699 0.01834 0.0135" rpy="${pi/2} ${pi} 2.3057"/>
-                <mass value=".00455"/>
-                <inertia ixx="0" ixy="0" ixz="0" iyy="0.000001" iyz="0" izz="0.000001"/>
-            </inertial>
-            <visual>
-                <origin xyz="-0.01699 0.01834 0.0135" rpy="${pi/2} ${pi} 2.3057"/>
-                <geometry>
-                    <mesh filename="package://bbot_description/meshes/gripper_link2.stl" scale="0.001 0.001 0.001"/>
-                </geometry>
-                <material name="Orange"/>
-            </visual>
-            <collision>
-                <origin xyz="-0.01699 0.01834 0.0135" rpy="${pi/2} ${pi} 2.3057"/>
-                <geometry>
-                    <mesh filename="package://bbot_description/meshes/gripper_link2.stl" scale="0.001 0.001 0.001"/>
                 </geometry>
                 <material name="Orange"/>
