Commit message: Added mimic joints to gripper ends

File: bbot_description/urdf/bbot.gazebo.xacro (robot description, xacro)
@@ -8,14 +8,4 @@
             </plugin>
         </gazebo>
-        <!-- Load Closed Loop Plug-in -->
-<!--         <gazebo>
-       <plugin name="Myrobot_ClosedLoopPlugin" filename="libpegasus_gazebo_closed_loop_plugin.so">
-           <joint>${robot_name}_joint_claw1_claw1_end_2</joint>
-           <child>${robot_name}_link_claw1_end</child>
-           <parent>${robot_name}_link_claw1_2</parent>
-           <position>-0.03678 -0.03387 0</position>
-           <rotation>0.00 0.00 0.00</rotation>
-       </plugin>
-        </gazebo> -->
         <!-- Link0 -->
         <gazebo reference="${robot_name}_link_baseplate">

File: bbot_description/urdf/bbot.xacro (robot description, xacro)
@@ -527,10 +527,22 @@
             has_pid="false" multiplier="-1.0" max_effort="${max_effort}" />
         <!-- joint between link_claw1 and link_claw1_end-->
-        <joint name="${robot_name}_joint_claw1_claw1_end" type="continuous">
+        <joint name="${robot_name}_joint_claw1_claw1_end" type="revolute">
             <parent link="${robot_name}_link_claw1"/>
             <child link="${robot_name}_link_claw1_end"/>
             <origin xyz="-0.03858 -0.03487 0" rpy="0 0 0"/>
             <axis xyz="0 0 1"/>
-        </joint>
+            <limit lower="${-170 * pi / 180}" upper="${170 * pi / 180}"
+                effort="${max_effort}" velocity="${max_velocity}" />
+            <safety_controller soft_lower_limit="${-168 * pi / 180}"
+                     soft_upper_limit="${168 * pi / 180}"
+                     k_position="${safety_controller_k_pos}"
+                     k_velocity="${safety_controller_k_vel}"/>
+            <dynamics damping="${joint_damping}"/>
+            <mimic joint="${robot_name}_joint_7" multiplier="1.0" offset = "0"/>
+        </joint>
+        <xacro:mimic_joint_plugin_gazebo name_prefix="${robot_name}_joint_claw1_claw1_end"
+            parent_joint="${robot_name}_joint_7"
+            mimic_joint="${robot_name}_joint_claw1_claw1_end"
+            has_pid="false" multiplier="-1.0" max_effort="${max_effort}" />
         <!-- link_claw1_end -->
         <link name="${robot_name}_link_claw1_end">
@@ -555,10 +567,4 @@
             </collision>
         </link>
-<!--         <joint name="${robot_name}_joint_claw1_claw1_end_2" type="continuous">
-            <parent link="${robot_name}_link_claw1_2"/>
-            <child link="${robot_name}_link_claw1_end"/>
-            <origin xyz="-0.03678 -0.03387 0" rpy="0 0 0"/>
-            <axis xyz="0 0 1"/>
-        </joint> -->
         <!-- link_claw2 -->
         <link name="${robot_name}_link_claw2">
@@ -630,5 +636,17 @@
             <origin xyz="0.03581 -0.0377 0" rpy="0 0 0"/>
             <axis xyz="0 0 1"/>
-        </joint>
+            <limit lower="${-170 * pi / 180}" upper="${170 * pi / 180}"
+                effort="${max_effort}" velocity="${max_velocity}" />
+            <safety_controller soft_lower_limit="${-168 * pi / 180}"
+                     soft_upper_limit="${168 * pi / 180}"
+                     k_position="${safety_controller_k_pos}"
+                     k_velocity="${safety_controller_k_vel}"/>
+            <dynamics damping="${joint_damping}"/>
+            <mimic joint="${robot_name}_joint_7" multiplier="1.0" offset = "0"/>
+        </joint>
+        <xacro:mimic_joint_plugin_gazebo name_prefix="${robot_name}_joint_claw2_claw2_end"
+            parent_joint="${robot_name}_joint_7"
+            mimic_joint="${robot_name}_joint_claw2_claw2_end"
+            has_pid="false" multiplier="1.0" max_effort="${max_effort}" />
         <!-- link_claw2_end -->
         <link name="${robot_name}_link_claw2_end">

Commit message: Made new testing branch for comparing Sim and real without gripper

File: bbot_description/urdf/bbot.gazebo.xacro (robot description, xacro)
@@ -80,5 +80,5 @@
             <mu2>0.2</mu2>
         </gazebo>
-        <gazebo reference="${robot_name}_link_motor7">
+        <!-- <gazebo reference="${robot_name}_link_motor7">
             <material>Gazebo/Black</material>
             <mu1>0.2</mu1>
@@ -114,5 +114,5 @@
             <mu1>0.2</mu1>
             <mu2>0.2</mu2>
-        </gazebo>
+        </gazebo> -->
     </xacro:macro>
     <!-- Load in mimic_joint_plugin -->

File: bbot_description/urdf/bbot.transmission.xacro (robot description, xacro)
@@ -68,5 +68,5 @@
       </actuator>
     </transmission>
-    <transmission name="${robot_name}_tran_7">
+    <!-- <transmission name="${robot_name}_tran_7">
       <robotNamespace>/${robot_name}</robotNamespace>
       <type>transmission_interface/SimpleTransmission</type>
@@ -78,5 +78,5 @@
         <mechanicalReduction>1</mechanicalReduction>
       </actuator>
-    </transmission>
+    </transmission> -->
   </xacro:macro>
 </robot>

File: bbot_description/urdf/bbot.xacro (robot description, xacro)
@@ -381,5 +381,5 @@
             <origin xyz="0 0 0.015" rpy="0 0 0"/>
         </joint>
-       <!-- link gripper_palm -->
+        <!-- link gripper_palm -->
         <link name="${robot_name}_gripper_palm">
             <inertial>
@@ -404,11 +404,11 @@
         </link>
         <!-- joint between gripper_palm and motor7 -->
-        <joint name="${robot_name}_joint_gripper_palm_motor7" type="fixed">
+        <!-- <joint name="${robot_name}_joint_gripper_palm_motor7" type="fixed">
             <parent link="${robot_name}_gripper_palm"/>
             <child link="${robot_name}_link_motor7"/>
             <origin xyz="-0.0305 -0.0065 0.0215" rpy="0 0 0"/>
-        </joint>
+        </joint> -->
         <!-- motor 7 -->
-        <link name="${robot_name}_link_motor7">
+        <!-- <link name="${robot_name}_link_motor7">
             <inertial>
                 <origin xyz="0.015 -0.0115 0.0295" rpy="${pi/2} 0 ${pi}"/>
@@ -430,7 +430,7 @@
                 <material name="Black"/>
             </collision>
-        </link>
+        </link> -->
         <!-- joint between motor 7 and link_claw1-->
-        <joint name="${robot_name}_joint_7" type="revolute">
+        <!-- <joint name="${robot_name}_joint_7" type="revolute">
             <parent link="${robot_name}_link_motor7"/>
             <child link="${robot_name}_link_claw1"/>
@@ -444,7 +444,7 @@
                      k_velocity="${safety_controller_k_vel}"/>
             <dynamics damping="${joint_damping}"/>
-        </joint>
+        </joint> -->
         <!-- link_claw1 -->
-        <link name="${robot_name}_link_claw1">
+        <!-- <link name="${robot_name}_link_claw1">
             <inertial>
                 <origin xyz="0 0 0" rpy="0 0 ${pi}"/>
@@ -466,7 +466,7 @@
                 <material name="Orange"/>
             </collision>
-        </link>
+        </link> -->
         <!-- joint between link_claw1 and link_claw1_2-->
-        <joint name="${robot_name}_joint_claw1_claw1_2" type="revolute">
+        <!-- <joint name="${robot_name}_joint_claw1_claw1_2" type="revolute">
             <parent link="${robot_name}_link_claw1"/>
             <child link="${robot_name}_link_claw1_2"/>
@@ -485,7 +485,7 @@
             parent_joint="${robot_name}_joint_7"
             mimic_joint="${robot_name}_joint_claw1_claw1_2"
-            has_pid="false" multiplier="1.0" max_effort="${max_effort}" />
+            has_pid="false" multiplier="1.0" max_effort="${max_effort}" /> -->
         <!-- link_claw1_2 -->
-        <link name="${robot_name}_link_claw1_2">
+        <!-- <link name="${robot_name}_link_claw1_2">
             <inertial>
                 <origin xyz="-0.01839 -0.01693 0.005" rpy="${-pi/2} 0 -2.3057"/>
@@ -507,7 +507,7 @@
                 <material name="Orange"/>
             </collision>
-        </link>
+        </link> -->
         <!-- joint between link_claw1 and link_claw2-->
-        <joint name="${robot_name}_joint_claw1_claw2" type="revolute">
+        <!-- <joint name="${robot_name}_joint_claw1_claw2" type="revolute">
             <parent link="${robot_name}_link_claw1"/>
             <child link="${robot_name}_link_claw2"/>
@@ -527,6 +527,7 @@
             mimic_joint="${robot_name}_joint_claw1_claw2"
             has_pid="false" multiplier="-1.0" max_effort="${max_effort}" />
+ -->
         <!-- joint between link_claw1 and link_claw1_end-->
-        <joint name="${robot_name}_joint_claw1_claw1_end" type="revolute">
+        <!-- <joint name="${robot_name}_joint_claw1_claw1_end" type="revolute">
             <parent link="${robot_name}_link_claw1"/>
             <child link="${robot_name}_link_claw1_end"/>
@@ -545,7 +546,7 @@
             parent_joint="${robot_name}_joint_7"
             mimic_joint="${robot_name}_joint_claw1_claw1_end"
-            has_pid="false" multiplier="-1.0" max_effort="${max_effort}" />
+            has_pid="false" multiplier="-1.0" max_effort="${max_effort}" /> -->
         <!-- link_claw1_end -->
-        <link name="${robot_name}_link_claw1_end">
+        <!-- <link name="${robot_name}_link_claw1_end">
             <inertial>
                 <origin xyz="0.01175 -0.0276 -0.005" rpy="${pi/2} 0 1.903"/>
@@ -567,7 +568,7 @@
                 <material name="Orange"/>
             </collision>
-        </link>
+        </link> -->
         <!-- link_claw2 -->
-        <link name="${robot_name}_link_claw2">
+        <!-- <link name="${robot_name}_link_claw2">
             <inertial>
                 <origin xyz="0 0 0.005" rpy="0 ${pi} 3.307"/>
@@ -589,7 +590,7 @@
                 <material name="Orange"/>
             </collision>
-        </link>
+        </link> -->
         <!-- joint between link_claw2 and link_claw2_2-->
-        <joint name="${robot_name}_joint_claw2_claw2_2" type="revolute">
+        <!-- <joint name="${robot_name}_joint_claw2_claw2_2" type="revolute">
             <parent link="${robot_name}_link_claw2"/>
             <child link="${robot_name}_link_claw2_2"/>
@@ -608,7 +609,7 @@
             parent_joint="${robot_name}_joint_7"
             mimic_joint="${robot_name}_joint_claw2_claw2_2"
-            has_pid="false" multiplier="-1.0" max_effort="${max_effort}" />
+            has_pid="false" multiplier="-1.0" max_effort="${max_effort}" /> -->
         <!-- link_claw2_2 -->
-        <link name="${robot_name}_link_claw2_2">
+        <!-- <link name="${robot_name}_link_claw2_2">
             <inertial>
                 <origin xyz="0.01699 -0.01834 0.005" rpy="${pi/2} ${pi} 2.3057"/>
@@ -630,7 +631,7 @@
                 <material name="Orange"/>
             </collision>
-        </link>
+        </link> -->
         <!-- joint between link_claw2 and link_claw2_end-->
-        <joint name="${robot_name}_joint_claw2_claw2_end" type="revolute">
+        <!-- <joint name="${robot_name}_joint_claw2_claw2_end" type="revolute">
             <parent link="${robot_name}_link_claw2"/>
             <child link="${robot_name}_link_claw2_end"/>
@@ -649,7 +650,7 @@
             parent_joint="${robot_name}_joint_7"
             mimic_joint="${robot_name}_joint_claw2_claw2_end"
-            has_pid="false" multiplier="1.0" max_effort="${max_effort}" />
+            has_pid="false" multiplier="1.0" max_effort="${max_effort}" /> -->
         <!-- link_claw2_end -->
-        <link name="${robot_name}_link_claw2_end">
+        <!-- <link name="${robot_name}_link_claw2_end">
             <inertial>
                 <origin xyz="-0.01181 -0.02758 0" rpy="${pi/2} ${pi} -1.903"/>
@@ -671,5 +672,5 @@
                 <material name="Orange"/>
             </collision>
-        </link>
+        </link> -->
         <xacro:bbot_gazebo robot_name="${robot_name}"/>
         <xacro:bbot_transmission hardware_interface="${hardware_interface}"/>
