Commit message: Put all the motors and links in place except the gripper.

File: bbot_description/urdf/bbot.xacro (robot description, xacro)
@@ -42,14 +42,14 @@
             <parent link="${robot_name}_link_baseplate"/>
             <child link="${robot_name}_link_motor1"/>
-            <origin xyz="0 0 0.01" rpy="0 0 0"/>
+            <origin xyz="0 0 0.0264" rpy="0 0 0"/>
         </joint>
         <link name="${robot_name}_link_motor1">
             <inertial>
-                <origin xyz="0 0 0.01" rpy="0 0 ${pi/2.0}"/>
+                <origin xyz="0 0 0" rpy="0 0 ${pi/2.0}"/>
                 <mass value="1"/>
                 <inertia ixx="0.000031" ixy="0" ixz="0" iyy="0.000013" iyz="0" izz="0.000027"/>
             </inertial>
             <visual>
-                <origin xyz="0 0 0.01" rpy="0 0 ${pi/2.0}"/>
+                <origin xyz="0 0 0" rpy="0 0 ${pi/2.0}"/>
                 <geometry>
                     <mesh filename="package://bbot_description/meshes/motor_no_idler.stl" scale="0.001 0.001 0.001"/>
@@ -58,5 +58,5 @@
             </visual>
             <collision>
-                <origin xyz="0 0 0.01" rpy="0 0 ${pi/2.0}"/>
+                <origin xyz="0 0 0" rpy="0 0 ${pi/2.0}"/>
                 <geometry>
                     <mesh filename="package://bbot_description/meshes/motor_no_idler.stl" scale="0.001 0.001 0.001"/>
@@ -68,5 +68,5 @@
             <parent link="${robot_name}_link_motor1"/>
             <child link="${robot_name}_link1_2"/>
-            <origin xyz="0 0 0.0517" rpy="0 0 0"/>
+            <origin xyz="0 0 0.0205" rpy="0 0 0"/>
             <axis xyz="0 0 1"/>
             <limit lower="${-170 * pi / 180}" upper="${170 * pi / 180}"
@@ -102,5 +102,5 @@
             <parent link="${robot_name}_link1_2"/>
             <child link="${robot_name}_link_motor2"/>
-            <origin xyz="0 0 0.1" rpy="${pi/2.0} ${-pi/2.0} 0"/>
+            <origin xyz="0 0 0.045" rpy="${pi/2.0} ${-pi/2.0} 0"/>
         </joint>
         <link name="${robot_name}_link_motor2">
@@ -140,10 +140,10 @@
         <link name="${robot_name}_link2_3">
             <inertial>
-                <origin xyz="0.1 0 0" rpy="${pi/2.0} ${-pi/2.0} 0"/>
-                <mass value="1"/>
-                <inertia ixx="1.0" ixy="0" ixz="0" iyy="1" iyz="0" izz="1"/>
-            </inertial>
-            <visual>
-                <origin xyz="0.1 0 0" rpy="${pi/2.0} ${-pi/2.0} 0"/>
+                <origin xyz="0.0275 0 0" rpy="${pi/2.0} ${-pi/2.0} 0"/>
+                <mass value="1"/>
+                <inertia ixx="1.0" ixy="0" ixz="0" iyy="1" iyz="0" izz="1"/>
+            </inertial>
+            <visual>
+                <origin xyz="0.0275 0 0" rpy="${pi/2.0} ${-pi/2.0} 0"/>
                 <geometry>
                     <mesh filename="package://bbot_description/meshes/link2_3.stl" scale="0.001 0.001 0.001"/>
@@ -152,5 +152,5 @@
             </visual>
             <collision>
-                <origin xyz="0.1 0 0" rpy="${pi/2.0} ${-pi/2.0} 0"/>
+                <origin xyz="0.0275 0 0" rpy="${pi/2.0} ${-pi/2.0} 0"/>
                 <geometry>
                     <mesh filename="package://bbot_description/meshes/link2_3.stl" scale="0.001 0.001 0.001"/>
@@ -162,5 +162,5 @@
             <parent link="${robot_name}_link2_3"/>
             <child link="${robot_name}_link_motor3"/>
-            <origin xyz="0.2 0 0" rpy="0 0 0"/>
+            <origin xyz="0.105 0 0" rpy="0 0 0"/>
             <axis xyz="0 0 1"/>
             <limit lower="${-170 * pi / 180}" upper="${170 * pi / 180}"
@@ -200,10 +200,10 @@
         <link name="${robot_name}_link3_4">
             <inertial>
-                <origin xyz="0.1 0 0" rpy="0 0 0"/>
-                <mass value="1"/>
-                <inertia ixx="1.0" ixy="0" ixz="0" iyy="1" iyz="0" izz="1"/>
-            </inertial>
-            <visual>
-                <origin xyz="0.1 0 0" rpy="0 0 0"/>
+                <origin xyz="0.067 0 0.01" rpy="0 0 0"/>
+                <mass value="1"/>
+                <inertia ixx="1.0" ixy="0" ixz="0" iyy="1" iyz="0" izz="1"/>
+            </inertial>
+            <visual>
+                <origin xyz="0.067 0 0.01" rpy="0 0 0"/>
                 <geometry>
                     <mesh filename="package://bbot_description/meshes/link3_4.stl" scale="0.001 0.001 0.001"/>
@@ -212,5 +212,5 @@
             </visual>
             <collision>
-                <origin xyz="0.1 0 0" rpy="0 0 0"/>
+                <origin xyz="0.067 0 0.01" rpy="0 0 0"/>
                 <geometry>
                     <mesh filename="package://bbot_description/meshes/link3_4.stl" scale="0.001 0.001 0.001"/>
@@ -222,21 +222,21 @@
             <parent link="${robot_name}_link3_4"/>
             <child link="${robot_name}_link_motor4"/>
-            <origin xyz="0.2 0 0" rpy="0 0 0"/>
+            <origin xyz="0.134 0 0" rpy="0 0 0"/>
         </joint>
         <link name="${robot_name}_link_motor4">
             <inertial>
-                <origin xyz="0 0 0" rpy="0 0 ${pi/2.0}"/>
-                <mass value="1"/>
-                <inertia ixx="1.0" ixy="0" ixz="0" iyy="1" iyz="0" izz="1"/>
-            </inertial>
-            <visual>
-                <origin xyz="0 0 0" rpy="0 0 ${pi/2.0}"/>
-                <geometry>
-                    <mesh filename="package://bbot_description/meshes/motor_with_idler.stl" scale="0.001 0.001 0.001"/>
-                </geometry>
-                <material name="Black"/>
-            </visual>
-            <collision>
-                <origin xyz="0 0 0" rpy="0 0 ${pi/2.0}"/>
+                <origin xyz="0 0 0" rpy="0 0 ${-pi/2.0}"/>
+                <mass value="1"/>
+                <inertia ixx="1.0" ixy="0" ixz="0" iyy="1" iyz="0" izz="1"/>
+            </inertial>
+            <visual>
+                <origin xyz="0 0 0" rpy="0 0 ${-pi/2.0}"/>
+                <geometry>
+                    <mesh filename="package://bbot_description/meshes/motor_with_idler.stl" scale="0.001 0.001 0.001"/>
+                </geometry>
+                <material name="Black"/>
+            </visual>
+            <collision>
+                <origin xyz="0 0 0" rpy="0 0 ${-pi/2.0}"/>
                 <geometry>
                     <mesh filename="package://bbot_description/meshes/motor_with_idler.stl" scale="0.001 0.001 0.001"/>
@@ -260,10 +260,10 @@
         <link name="${robot_name}_link4_5">
             <inertial>
-                <origin xyz="0 0 0.1" rpy="0 0 0"/>
-                <mass value="1"/>
-                <inertia ixx="1.0" ixy="0" ixz="0" iyy="1" iyz="0" izz="1"/>
-            </inertial>
-            <visual>
-                <origin xyz="0 0 0.1" rpy="0 0 0"/>
+                <origin xyz="0 0 0.0235" rpy="0 0 0"/>
+                <mass value="1"/>
+                <inertia ixx="1.0" ixy="0" ixz="0" iyy="1" iyz="0" izz="1"/>
+            </inertial>
+            <visual>
+                <origin xyz="0 0 0.0235" rpy="0 0 0"/>
                 <geometry>
                     <mesh filename="package://bbot_description/meshes/link4_5.stl" scale="0.001 0.001 0.001"/>
@@ -272,5 +272,5 @@
             </visual>
             <collision>
-                <origin xyz="0 0 0.1" rpy="0 0 0"/>
+                <origin xyz="0 0 0.0235" rpy="0 0 0"/>
                 <geometry>
                     <mesh filename="package://bbot_description/meshes/link4_5.stl" scale="0.001 0.001 0.001"/>
@@ -282,5 +282,5 @@
             <parent link="${robot_name}_link4_5"/>
             <child link="${robot_name}_link_motor5"/>
-            <origin xyz="0 0 0.15" rpy="${pi/2.0} ${-pi/2.0} 0"/>
+            <origin xyz="0 0 0.0625" rpy="${pi/2.0} ${-pi/2.0} 0"/>
             <axis xyz="0 0 1"/>
             <limit lower="${-170 * pi / 180}" upper="${170 * pi / 180}"
@@ -316,14 +316,14 @@
             <parent link="${robot_name}_link_motor5"/>
             <child link="${robot_name}_link5_6"/>
-            <origin xyz="0 -0.1 0" rpy="0 0 0"/>
+            <origin xyz="0 -0.0371 0" rpy="0 0 0"/>
         </joint>
         <link name="${robot_name}_link5_6">
             <inertial>
-                <origin xyz="0 0 0" rpy="${pi/2.0} 0 ${pi/2.0}"/>
-                <mass value="1"/>
-                <inertia ixx="1.0" ixy="0" ixz="0" iyy="1" iyz="0" izz="1"/>
-            </inertial>
-            <visual>
-                <origin xyz="0 0 0" rpy="${pi/2.0} 0 ${pi/2.0}"/>
+                <origin xyz="0 0 0.0173" rpy="${pi/2.0} 0 ${pi/2.0}"/>
+                <mass value="1"/>
+                <inertia ixx="1.0" ixy="0" ixz="0" iyy="1" iyz="0" izz="1"/>
+            </inertial>
+            <visual>
+                <origin xyz="0 0 0.0173" rpy="${pi/2.0} 0 ${pi/2.0}"/>
                 <geometry>
                     <mesh filename="package://bbot_description/meshes/link5_6.stl" scale="0.001 0.001 0.001"/>
@@ -332,5 +332,5 @@
             </visual>
             <collision>
-                <origin xyz="0 0 0" rpy="${pi/2.0} 0 ${pi/2.0}"/>
+                <origin xyz="0 0 0.0173" rpy="${pi/2.0} 0 ${pi/2.0}"/>
                 <geometry>
                     <mesh filename="package://bbot_description/meshes/link5_6.stl" scale="0.001 0.001 0.001"/>
@@ -342,5 +342,5 @@
             <parent link="${robot_name}_link5_6"/>
             <child link="${robot_name}_link_motor6"/>
-            <origin xyz="0 -0.1 0" rpy="${pi/2.0} 0 0"/>
+            <origin xyz="0 -0.0332 0" rpy="${pi/2.0} 0 0"/>
             <axis xyz="0 0 1"/>
             <limit lower="${-170 * pi / 180}" upper="${170 * pi / 180}"

Commit message: Updated joint names

File: bbot_description/urdf/bbot.xacro (robot description, xacro)
@@ -66,5 +66,5 @@
             </collision>
         </link>
-        <joint name="${robot_name}_joint_motor1_link1_2" type="revolute">
+        <joint name="${robot_name}_joint_1" type="revolute">
             <parent link="${robot_name}_link_motor1"/>
             <child link="${robot_name}_link1_2"/>
@@ -126,5 +126,5 @@
             </collision>
         </link>
-        <joint name="${robot_name}_joint_motor2_link2_3" type="revolute">
+        <joint name="${robot_name}_joint_2" type="revolute">
             <parent link="${robot_name}_link_motor2"/>
             <child link="${robot_name}_link2_3"/>
@@ -160,5 +160,5 @@
             </collision>
         </link>
-        <joint name="${robot_name}_joint_link2_3_motor3" type="revolute">
+        <joint name="${robot_name}_joint_3" type="revolute">
             <parent link="${robot_name}_link2_3"/>
             <child link="${robot_name}_link_motor3"/>
@@ -246,5 +246,5 @@
             </collision>
         </link>
-        <joint name="${robot_name}_joint_motor4_link4_5" type="revolute">
+        <joint name="${robot_name}_joint_4" type="revolute">
             <parent link="${robot_name}_link_motor4"/>
             <child link="${robot_name}_link4_5"/>
@@ -280,5 +280,5 @@
             </collision>
         </link>
-        <joint name="${robot_name}_joint_link4_5_motor5" type="revolute">
+        <joint name="${robot_name}_joint_5" type="revolute">
             <parent link="${robot_name}_link4_5"/>
             <child link="${robot_name}_link_motor5"/>
@@ -340,5 +340,5 @@
             </collision>
         </link>
-        <joint name="${robot_name}_joint_link5_6_motor6" type="revolute">
+        <joint name="${robot_name}_joint_6" type="revolute">
             <parent link="${robot_name}_link5_6"/>
             <child link="${robot_name}_link_motor6"/>
@@ -374,8 +374,4 @@
             </collision>
         </link>
-        <!-- joint between motor 5 and link 5_6 -->
-        <!-- link 5_6 -->
-        <!-- joint between link 5_6 and motor6 -->
-        <!-- motor 6 -->
         <!-- joint between motor6 and link_grasper_base-->
         <!-- link_grasper_base -->

Commit message: Added inertia/mass values. In process of adding gripper info

File: bbot_description/urdf/bbot.xacro (robot description, xacro)
@@ -22,5 +22,5 @@
             <inertial>
                 <origin xyz="0 0 0" rpy="${pi/2.0} 0 0"/>
-                <mass value="1"/>
+                <mass value="0.0800"/>
                 <inertia ixx="0.000070" ixy="0" ixz="0" iyy="0.000174" iyz="0" izz="0.000107"/>
             </inertial>
@@ -48,5 +48,5 @@
             <inertial>
                 <origin xyz="0 0 0" rpy="0 0 ${pi/2.0}"/>
-                <mass value="1"/>
+                <mass value="0.074"/>
                 <inertia ixx="0.000031" ixy="0" ixz="0" iyy="0.000013" iyz="0" izz="0.000027"/>
             </inertial>
@@ -82,6 +82,6 @@
             <inertial>
                 <origin xyz="0 0 0" rpy="${pi/2.0} 0 ${pi/2.0}"/>
-                <mass value="1"/>
-                <inertia ixx="1.0" ixy="0" ixz="0" iyy="1" iyz="0" izz="1"/>
+                <mass value="0.0296"/>
+                <inertia ixx="0.000028" ixy="0" ixz="0" iyy="0.000014" iyz="0" izz="0.000023"/>
             </inertial>
             <visual>
@@ -108,6 +108,6 @@
             <inertial>
                 <origin xyz="0 0 0" rpy="0 0 ${-pi/2.0}"/>
-                <mass value="1"/>
-                <inertia ixx="1.0" ixy="0" ixz="0" iyy="1" iyz="0" izz="1"/>
+                <mass value="0.076"/>
+                <inertia ixx="0.000031" ixy="0" ixz="0" iyy="0.000014" iyz="0" izz="0.000018"/>
             </inertial>
             <visual>
@@ -142,6 +142,6 @@
             <inertial>
                 <origin xyz="0.0275 0 0" rpy="${pi/2.0} ${-pi/2.0} 0"/>
-                <mass value="1"/>
-                <inertia ixx="1.0" ixy="0" ixz="0" iyy="1" iyz="0" izz="1"/>
+                <mass value="0.0584"/>
+                <inertia ixx="0.000096" ixy="0" ixz="0" iyy="0.000021" iyz="0" izz="0.00011"/>
             </inertial>
             <visual>
@@ -176,6 +176,6 @@
             <inertial>
                 <origin xyz="0 0 0" rpy="0 0 ${pi/2.0}"/>
-                <mass value="1"/>
-                <inertia ixx="1.0" ixy="0" ixz="0" iyy="1" iyz="0" izz="1"/>
+                <mass value="0.076"/>
+                <inertia ixx="0.000031" ixy="0" ixz="0" iyy="0.000014" iyz="0" izz="0.000027"/>
             </inertial>
             <visual>
@@ -202,6 +202,6 @@
             <inertial>
                 <origin xyz="0.067 0 0.01" rpy="0 0 0"/>
-                <mass value="1"/>
-                <inertia ixx="1.0" ixy="0" ixz="0" iyy="1" iyz="0" izz="1"/>
+                <mass value="0.0409"/>
+                <inertia ixx="0.000016" ixy="0" ixz="0" iyy="0.000053" iyz="0" izz="0.000049"/>
             </inertial>
             <visual>
@@ -228,6 +228,6 @@
             <inertial>
                 <origin xyz="0 0 0" rpy="0 0 ${-pi/2.0}"/>
-                <mass value="1"/>
-                <inertia ixx="1.0" ixy="0" ixz="0" iyy="1" iyz="0" izz="1"/>
+                <mass value="0.076"/>
+                <inertia ixx="0.000031" ixy="0" ixz="0" iyy="0.000014" iyz="0" izz="0.000027"/>
             </inertial>
             <visual>
@@ -262,6 +262,6 @@
             <inertial>
                 <origin xyz="0 0 0.0235" rpy="0 0 0"/>
-                <mass value="1"/>
-                <inertia ixx="1.0" ixy="0" ixz="0" iyy="1" iyz="0" izz="1"/>
+                <mass value="0.021"/>
+                <inertia ixx="0.000016" ixy="0" ixz="0" iyy="0.000008" iyz="0" izz="0.00001"/>
             </inertial>
             <visual>
@@ -296,6 +296,6 @@
             <inertial>
                 <origin xyz="0 0 0" rpy="0 0 0"/>
-                <mass value="1"/>
-                <inertia ixx="1.0" ixy="0" ixz="0" iyy="1" iyz="0" izz="1"/>
+                <mass value="0.076"/>
+                <inertia ixx="0.000031" ixy="0" ixz="0" iyy="0.000014" iyz="0" izz="0.000027"/>
             </inertial>
             <visual>
@@ -322,6 +322,6 @@
             <inertial>
                 <origin xyz="0 0 0.0173" rpy="${pi/2.0} 0 ${pi/2.0}"/>
-                <mass value="1"/>
-                <inertia ixx="1.0" ixy="0" ixz="0" iyy="1" iyz="0" izz="1"/>
+                <mass value="0.01588"/>
+                <inertia ixx="0.00001" ixy="0" ixz="0" iyy="0.000003" iyz="0" izz="0.000009"/>
             </inertial>
             <visual>
@@ -356,26 +356,78 @@
             <inertial>
                 <origin xyz="0 0 0" rpy="0 0 ${pi}"/>
-                <mass value="1"/>
-                <inertia ixx="1.0" ixy="0" ixz="0" iyy="1" iyz="0" izz="1"/>
-            </inertial>
-            <visual>
-                <origin xyz="0 0 0" rpy="0 0 ${pi}"/>
-                <geometry>
-                    <mesh filename="package://bbot_description/meshes/motor_with_idler.stl" scale="0.001 0.001 0.001"/>
-                </geometry>
-                <material name="Black"/>
-            </visual>
-            <collision>
-                <origin xyz="0 0 0" rpy="0 0 ${pi}"/>
-                <geometry>
-                    <mesh filename="package://bbot_description/meshes/motor_with_idler.stl" scale="0.001 0.001 0.001"/>
-                </geometry>
-                <material name="Black"/>
-            </collision>
-        </link>
-        <!-- joint between motor6 and link_grasper_base-->
-        <!-- link_grasper_base -->
-        <!-- joint between link_grasper_base and motor7 -->
+                <mass value="0.076"/>
+                <inertia ixx="0.000031" ixy="0" ixz="0" iyy="0.000014" iyz="0" izz="0.000027"/>
+            </inertial>
+            <visual>
+                <origin xyz="0 0 0" rpy="0 0 ${pi}"/>
+                <geometry>
+                    <mesh filename="package://bbot_description/meshes/motor_with_idler.stl" scale="0.001 0.001 0.001"/>
+                </geometry>
+                <material name="Black"/>
+            </visual>
+            <collision>
+                <origin xyz="0 0 0" rpy="0 0 ${pi}"/>
+                <geometry>
+                    <mesh filename="package://bbot_description/meshes/motor_with_idler.stl" scale="0.001 0.001 0.001"/>
+                </geometry>
+                <material name="Black"/>
+            </collision>
+        </link>
+        <!-- joint between motor6 and gripper_palm-->
+        <joint name="${robot_name}_joint_motor6_gripper_palm" type="fixed">
+            <parent link="${robot_name}_link_motor6"/>
+            <child link="${robot_name}_gripper_palm"/>
+            <origin xyz="0 0 0.015" rpy="0 0 0"/>
+        </joint>
+        <!-- link gripper_palm -->
+        <link name="${robot_name}_gripper_palm">
+            <inertial>
+                <origin xyz="0 0 0.0073" rpy="${pi} 0 ${0.0}"/>
+                <mass value="0.0646"/>
+                <inertia ixx="0.000077" ixy="0.000001" ixz="-0.000001" iyy="0.000086" iyz="-0.00001" izz="0.000024"/>
+            </inertial>
+            <visual>
+                <origin xyz="0 0 0.0073" rpy="${pi} 0 ${0.0}"/>
+                <geometry>
+                    <mesh filename="package://bbot_description/meshes/gripper_palm.stl" scale="0.001 0.001 0.001"/>
+                </geometry>
+                <material name="Orange"/>
+            </visual>
+            <collision>
+                <origin xyz="0 0 0.0073" rpy="${pi} 0 ${0.0}"/>
+                <geometry>
+                    <mesh filename="package://bbot_description/meshes/gripper_palm.stl" scale="0.001 0.001 0.001"/>
+                </geometry>
+                <material name="Orange"/>
+            </collision>
+        </link>
+        <!-- joint between gripper_palm and motor7 -->
+        <joint name="${robot_name}_joint_gripper_palm_motor7" type="fixed">
+            <parent link="${robot_name}_gripper_palm"/>
+            <child link="${robot_name}_link_motor7"/>
+            <origin xyz="0 0.2 0" rpy="0 0 0"/>
+        </joint>
         <!-- motor 7 -->
+        <link name="${robot_name}_link_motor7">
+            <inertial>
+                <origin xyz="0 0 0" rpy="0 0 ${pi}"/>
+                <mass value="0.076"/>
+                <inertia ixx="0.000031" ixy="0" ixz="0" iyy="0.000014" iyz="0" izz="0.000027"/>
+            </inertial>
+            <visual>
+                <origin xyz="0 0 0" rpy="0 0 ${pi}"/>
+                <geometry>
+                    <mesh filename="package://bbot_description/meshes/motor_with_idler.stl" scale="0.001 0.001 0.001"/>
+                </geometry>
+                <material name="Black"/>
+            </visual>
+            <collision>
+                <origin xyz="0 0 0" rpy="0 0 ${pi}"/>
+                <geometry>
+                    <mesh filename="package://bbot_description/meshes/motor_with_idler.stl" scale="0.001 0.001 0.001"/>
+                </geometry>
+                <material name="Black"/>
+            </collision>
+        </link>
         <!-- joint between motor 7 and link_claw1-->
         <!-- link_claw1 -->
