Commit message: Finished adding gripper to URDF

File: bbot_description/urdf/bbot.xacro (robot description, xacro)
@@ -475,10 +475,10 @@
         <link name="${robot_name}_link_claw1_end">
             <inertial>
-                <origin xyz="0.001179 -0.02759 0.00325" rpy="${pi/2} 0 ${0.6*pi}"/>
+                <origin xyz="0.01175 -0.0276 0.00325" rpy="${pi/2} 0 1.903"/>
                 <mass value="0.006"/>
                 <inertia ixx="0" ixy="0" ixz="0" iyy="0.000003" iyz="0" izz="0.000003"/>
             </inertial>
             <visual>
-                <origin xyz="0.001179 -0.02759 0.00325" rpy="${pi/2} 0 ${0.6*pi}"/>
+                <origin xyz="0.01175 -0.0276 0.00325" rpy="${pi/2} 0 1.903"/>
                 <geometry>
                     <mesh filename="package://bbot_description/meshes/gripper_link3.stl" scale="0.001 0.001 0.001"/>
@@ -487,5 +487,5 @@
             </visual>
             <collision>
-                <origin xyz="0.00179 -0.02759 0.00325" rpy="${pi/2} 0 ${0.6*pi}"/>
+                <origin xyz="0.01175 -0.0276 0.00325" rpy="${pi/2} 0 1.903"/>
                 <geometry>
                     <mesh filename="package://bbot_description/meshes/gripper_link3.stl" scale="0.001 0.001 0.001"/>
@@ -494,19 +494,47 @@
             </collision>
         </link>
+        <!-- joint between link_claw1_end and link_claw1_2-->
+        <joint name="${robot_name}_joint_claw1_end_claw1_2" type="fixed">
+            <parent link="${robot_name}_link_claw1_end"/>
+            <child link="${robot_name}_link_claw1_2"/>
+            <origin xyz="0.0098 -0.023 0.00025" rpy="0 0 0"/>
+        </joint>
+        <!-- link_claw1_2 -->
+        <link name="${robot_name}_link_claw1_2">
+            <inertial>
+                <origin xyz="0.01839 0.01693 0.0135" rpy="${-pi/2} 0 -2.3057"/>
+                <mass value=".00455"/>
+                <inertia ixx="0" ixy="0" ixz="0" iyy="0.000001" iyz="0" izz="0.000001"/>
+            </inertial>
+            <visual>
+                <origin xyz="0.01839 0.01693 0.0135" rpy="${-pi/2} 0 -2.3057"/>
+                <geometry>
+                    <mesh filename="package://bbot_description/meshes/gripper_link2.stl" scale="0.001 0.001 0.001"/>
+                </geometry>
+                <material name="Orange"/>
+            </visual>
+            <collision>
+                <origin xyz="0.01839 0.01693 0.0135" rpy="${-pi/2} 0 -2.3057"/>
+                <geometry>
+                    <mesh filename="package://bbot_description/meshes/gripper_link2.stl" scale="0.001 0.001 0.001"/>
+                </geometry>
+                <material name="Orange"/>
+            </collision>
+        </link>
         <!-- joint between link_claw1 and link_claw2-->
-<!--         <joint name="${robot_name}_joint_claw1_claw2" type="fixed">
+        <joint name="${robot_name}_joint_claw1_claw2" type="fixed">
             <parent link="${robot_name}_link_claw1"/>
             <child link="${robot_name}_link_claw2"/>
-            <origin xyz="0 0 0" rpy="0 0 0"/>
-        </joint> -->
-        <!-- link_claw2 -->
-<!--         <link name="${robot_name}_link_claw2">
-            <inertial>
-                <origin xyz="0 0 0" rpy="${pi/2} 0 0"/>
+            <origin xyz="0.03 0 0" rpy="0 0 0"/>
+        </joint>
+        <!-- link_claw2_2 -->
+        <link name="${robot_name}_link_claw2">
+            <inertial>
+                <origin xyz="0 0 0.005" rpy="0 ${pi} ${pi}"/>
                 <mass value=".0066"/>
-                <inertia ixx="0.000004" ixy="0.000001" ixz="0" iyy="0.000002" iyz="0.000001" izz="0.000006"/>
-            </inertial>
-            <visual>
-                <origin xyz="0 0 0" rpy="${pi/2} 0 0"/>
+                <inertia ixx="0.000004" ixy="0.000003" ixz="0" iyy="0.000002" iyz="0.000001" izz="0.000006"/>
+            </inertial>
+            <visual>
+                <origin xyz="0 0 0.005" rpy="0 ${pi} ${pi}"/>
                 <geometry>
                     <mesh filename="package://bbot_description/meshes/gripper_link1_left.stl" scale="0.001 0.001 0.001"/>
@@ -515,5 +543,5 @@
             </visual>
             <collision>
-                <origin xyz="0 0 0" rpy="${pi/2} 0 0"/>
+                <origin xyz="0 0 0.005" rpy="0 ${pi} ${pi}"/>
                 <geometry>
                     <mesh filename="package://bbot_description/meshes/gripper_link1_left.stl" scale="0.001 0.001 0.001"/>
@@ -521,20 +549,20 @@
                 <material name="Orange"/>
             </collision>
-        </link> -->
+        </link>
         <!-- joint between link_claw2 and link_claw2_end-->
-<!--         <joint name="${robot_name}_joint_claw2_claw2_end" type="fixed">
+        <joint name="${robot_name}_joint_claw2_claw2_end" type="fixed">
             <parent link="${robot_name}_link_claw2"/>
             <child link="${robot_name}_link_claw2_end"/>
-            <origin xyz="0 0 0" rpy="0 0 0"/>
-        </joint> -->
-        <!-- link_claw2_end -->
-<!--         <link name="${robot_name}_link_claw2_end">
-            <inertial>
-                <origin xyz="0 0 0" rpy="0 ${0.6*pi} ${pi}"/>
-                <mass value=".006"/>
+            <origin xyz="0.03581 -0.0377 -0.0085" rpy="0 0 0"/>
+        </joint>
+        <!-- link_claw1_end -->
+        <link name="${robot_name}_link_claw2_end">
+            <inertial>
+                <origin xyz="-0.01181 -0.02758 0.0085" rpy="${pi/2} ${pi} -1.903"/>
+                <mass value="0.006"/>
                 <inertia ixx="0" ixy="0" ixz="0" iyy="0.000003" iyz="0" izz="0.000003"/>
             </inertial>
             <visual>
-                <origin xyz="0 0 0" rpy="0 ${0.6*pi} ${pi}"/>
+                <origin xyz="-0.01181 -0.02758 0.0085" rpy="${pi/2} ${pi} -1.903"/>
                 <geometry>
                     <mesh filename="package://bbot_description/meshes/gripper_link3.stl" scale="0.001 0.001 0.001"/>
@@ -543,5 +571,5 @@
             </visual>
             <collision>
-                <origin xyz="0 0 0" rpy="0 ${0.6*pi} ${pi}"/>
+                <origin xyz="-0.01181 -0.02758 0.0085" rpy="${pi/2} ${pi} -1.903"/>
                 <geometry>
                     <mesh filename="package://bbot_description/meshes/gripper_link3.stl" scale="0.001 0.001 0.001"/>
@@ -549,5 +577,33 @@
                 <material name="Orange"/>
             </collision>
-        </link> -->
+        </link>
+        <!-- joint between link_claw2_end and link_claw2_2-->
+        <joint name="${robot_name}_joint_claw1_end_claw2_2" type="fixed">
+            <parent link="${robot_name}_link_claw2_end"/>
+            <child link="${robot_name}_link_claw2_2"/>
+            <origin xyz="-0.00984 -0.02298 0" rpy="0 0 0"/>
+        </joint>
+        <!-- link_claw2_2 -->
+        <link name="${robot_name}_link_claw2_2">
+            <inertial>
+                <origin xyz="-0.01699 0.01834 0.0135" rpy="${pi/2} ${pi} 2.3057"/>
+                <mass value=".00455"/>
+                <inertia ixx="0" ixy="0" ixz="0" iyy="0.000001" iyz="0" izz="0.000001"/>
+            </inertial>
+            <visual>
+                <origin xyz="-0.01699 0.01834 0.0135" rpy="${pi/2} ${pi} 2.3057"/>
+                <geometry>
+                    <mesh filename="package://bbot_description/meshes/gripper_link2.stl" scale="0.001 0.001 0.001"/>
+                </geometry>
+                <material name="Orange"/>
+            </visual>
+            <collision>
+                <origin xyz="-0.01699 0.01834 0.0135" rpy="${pi/2} ${pi} 2.3057"/>
+                <geometry>
+                    <mesh filename="package://bbot_description/meshes/gripper_link2.stl" scale="0.001 0.001 0.001"/>
+                </geometry>
+                <material name="Orange"/>
+            </collision>
+        </link>
         <xacro:bbot_gazebo robot_name="${robot_name}"/>
         <xacro:bbot_transmission hardware_interface="${hardware_interface}"/>

Commit message: Scrubbed all inertia and mass values

File: bbot_description/urdf/bbot.xacro (robot description, xacro)
@@ -109,5 +109,5 @@
                 <origin xyz="0 0 0" rpy="0 0 ${-pi/2.0}"/>
                 <mass value="0.076"/>
-                <inertia ixx="0.000031" ixy="0" ixz="0" iyy="0.000014" iyz="0" izz="0.000018"/>
+                <inertia ixx="0.000031" ixy="0" ixz="0" iyy="0.000014" iyz="0" izz="0.000027"/>
             </inertial>
             <visual>
@@ -203,5 +203,5 @@
                 <origin xyz="0.067 0 0.01" rpy="0 0 0"/>
                 <mass value="0.0409"/>
-                <inertia ixx="0.000016" ixy="0" ixz="0" iyy="0.000053" iyz="0" izz="0.000049"/>
+                <inertia ixx="0.0027" ixy="-0.0001" ixz="0" iyy="0" iyz="0" izz="0.0027"/>
             </inertial>
             <visual>
@@ -323,5 +323,5 @@
                 <origin xyz="0 0 0.0173" rpy="${pi/2.0} 0 ${pi/2.0}"/>
                 <mass value="0.01588"/>
-                <inertia ixx="0.00001" ixy="0" ixz="0" iyy="0.000003" iyz="0" izz="0.000009"/>
+                <inertia ixx="0.00001" ixy="0.000002" ixz="0" iyy="0.000003" iyz="0" izz="0.000009"/>
             </inertial>
             <visual>
@@ -385,5 +385,5 @@
                 <origin xyz="0 0.0175 0.008" rpy="${pi} 0 ${0.0}"/>
                 <mass value="0.07825"/>
-                <inertia ixx="0.00013" ixy="0" ixz="-0" iyy="0.00014" iyz="-0.00002" izz="0.00003"/>
+                <inertia ixx="0.00013" ixy="-0.000001" ixz="0" iyy="0.000141" iyz="-0.000015" izz="0.00003"/>
             </inertial>
             <visual>
@@ -467,11 +467,11 @@
         </link>
         <!-- joint between link_claw1 and link_claw1_end-->
-        <joint name="${robot_name}_joint_claw1_claw1_end" type="fixed">
+<!--         <joint name="${robot_name}_joint_claw1_claw1_end" type="fixed">
             <parent link="${robot_name}_link_claw1"/>
             <child link="${robot_name}_link_claw1_end"/>
             <origin xyz="-0.03677 -0.03677 -0.00825" rpy="0 0 0"/>
-        </joint>
+        </joint> -->
         <!-- link_claw1_end -->
-        <link name="${robot_name}_link_claw1_end">
+<!--         <link name="${robot_name}_link_claw1_end">
             <inertial>
                 <origin xyz="0.01175 -0.0276 0.00325" rpy="${pi/2} 0 1.903"/>
@@ -493,13 +493,13 @@
                 <material name="Orange"/>
             </collision>
-        </link>
+        </link> -->
         <!-- joint between link_claw1_end and link_claw1_2-->
-        <joint name="${robot_name}_joint_claw1_end_claw1_2" type="fixed">
+<!--         <joint name="${robot_name}_joint_claw1_end_claw1_2" type="fixed">
             <parent link="${robot_name}_link_claw1_end"/>
             <child link="${robot_name}_link_claw1_2"/>
             <origin xyz="0.0098 -0.023 0.00025" rpy="0 0 0"/>
-        </joint>
+        </joint> -->
         <!-- link_claw1_2 -->
-        <link name="${robot_name}_link_claw1_2">
+<!--         <link name="${robot_name}_link_claw1_2">
             <inertial>
                 <origin xyz="0.01839 0.01693 0.0135" rpy="${-pi/2} 0 -2.3057"/>
@@ -521,13 +521,13 @@
                 <material name="Orange"/>
             </collision>
-        </link>
+        </link> -->
         <!-- joint between link_claw1 and link_claw2-->
-        <joint name="${robot_name}_joint_claw1_claw2" type="fixed">
+<!--         <joint name="${robot_name}_joint_claw1_claw2" type="fixed">
             <parent link="${robot_name}_link_claw1"/>
             <child link="${robot_name}_link_claw2"/>
             <origin xyz="0.03 0 0" rpy="0 0 0"/>
-        </joint>
+        </joint> -->
         <!-- link_claw2_2 -->
-        <link name="${robot_name}_link_claw2">
+<!--         <link name="${robot_name}_link_claw2">
             <inertial>
                 <origin xyz="0 0 0.005" rpy="0 ${pi} ${pi}"/>
@@ -550,12 +550,13 @@
             </collision>
         </link>
+ -->
         <!-- joint between link_claw2 and link_claw2_end-->
-        <joint name="${robot_name}_joint_claw2_claw2_end" type="fixed">
+<!--         <joint name="${robot_name}_joint_claw2_claw2_end" type="fixed">
             <parent link="${robot_name}_link_claw2"/>
             <child link="${robot_name}_link_claw2_end"/>
             <origin xyz="0.03581 -0.0377 -0.0085" rpy="0 0 0"/>
-        </joint>
-        <!-- link_claw1_end -->
-        <link name="${robot_name}_link_claw2_end">
+        </joint> -->
+        <!-- link_claw2_end -->
+<!--         <link name="${robot_name}_link_claw2_end">
             <inertial>
                 <origin xyz="-0.01181 -0.02758 0.0085" rpy="${pi/2} ${pi} -1.903"/>
@@ -577,13 +578,13 @@
                 <material name="Orange"/>
             </collision>
-        </link>
+        </link> -->
         <!-- joint between link_claw2_end and link_claw2_2-->
-        <joint name="${robot_name}_joint_claw1_end_claw2_2" type="fixed">
+<!--         <joint name="${robot_name}_joint_claw1_end_claw2_2" type="fixed">
             <parent link="${robot_name}_link_claw2_end"/>
             <child link="${robot_name}_link_claw2_2"/>
             <origin xyz="-0.00984 -0.02298 0" rpy="0 0 0"/>
-        </joint>
+        </joint> -->
         <!-- link_claw2_2 -->
-        <link name="${robot_name}_link_claw2_2">
+<!--         <link name="${robot_name}_link_claw2_2">
             <inertial>
                 <origin xyz="-0.01699 0.01834 0.0135" rpy="${pi/2} ${pi} 2.3057"/>
@@ -605,5 +606,5 @@
                 <material name="Orange"/>
             </collision>
-        </link>
+        </link> -->
         <xacro:bbot_gazebo robot_name="${robot_name}"/>
         <xacro:bbot_transmission hardware_interface="${hardware_interface}"/>

Commit message: Added inner control loop config files

File: bbot_description/urdf/bbot.xacro (robot description, xacro)
@@ -467,11 +467,11 @@
         </link>
         <!-- joint between link_claw1 and link_claw1_end-->
-        <joint name="${robot_name}_joint_claw1_claw1_end" type="fixed">
+        <!-- <joint name="${robot_name}_joint_claw1_claw1_end" type="fixed">
             <parent link="${robot_name}_link_claw1"/>
             <child link="${robot_name}_link_claw1_end"/>
             <origin xyz="-0.03677 -0.03677 -0.00825" rpy="0 0 0"/>
-        </joint>
+        </joint> -->
         <!-- link_claw1_end -->
-        <link name="${robot_name}_link_claw1_end">
+        <!-- <link name="${robot_name}_link_claw1_end">
             <inertial>
                 <origin xyz="0.01175 -0.0276 0.00325" rpy="${pi/2} 0 1.903"/>
@@ -493,13 +493,13 @@
                 <material name="Orange"/>
             </collision>
-        </link>
+        </link> -->
         <!-- joint between link_claw1_end and link_claw1_2-->
-        <joint name="${robot_name}_joint_claw1_end_claw1_2" type="fixed">
+        <!-- <joint name="${robot_name}_joint_claw1_end_claw1_2" type="fixed">
             <parent link="${robot_name}_link_claw1_end"/>
             <child link="${robot_name}_link_claw1_2"/>
             <origin xyz="0.0098 -0.023 0.00025" rpy="0 0 0"/>
-        </joint>
+        </joint> -->
         <!-- link_claw1_2 -->
-        <link name="${robot_name}_link_claw1_2">
+        <!-- <link name="${robot_name}_link_claw1_2">
             <inertial>
                 <origin xyz="0.01839 0.01693 0.0135" rpy="${-pi/2} 0 -2.3057"/>
@@ -521,5 +521,5 @@
                 <material name="Orange"/>
             </collision>
-        </link>
+        </link> -->
         <!-- joint between link_claw1 and link_claw2-->
         <joint name="${robot_name}_joint_claw1_claw2" type="revolute">
@@ -540,5 +540,5 @@
             parent_joint="${robot_name}_joint_7"
             mimic_joint="${robot_name}_joint_claw1_claw2"
-            has_pid="true" multiplier="-1.0" max_effort="${max_effort}" />
+            has_pid="false" multiplier="-1.0" max_effort="${max_effort}" />
         <!-- link_claw2 -->
         <link name="${robot_name}_link_claw2">
@@ -564,11 +564,11 @@
         </link>
         <!-- joint between link_claw2 and link_claw2_end-->
-        <joint name="${robot_name}_joint_claw2_claw2_end" type="fixed">
+        <!-- <joint name="${robot_name}_joint_claw2_claw2_end" type="fixed">
             <parent link="${robot_name}_link_claw2"/>
             <child link="${robot_name}_link_claw2_end"/>
             <origin xyz="0.03581 -0.0377 -0.0085" rpy="0 0 0"/>
-        </joint>
+        </joint> -->
         <!-- link_claw2_end -->
-        <link name="${robot_name}_link_claw2_end">
+        <!-- <link name="${robot_name}_link_claw2_end">
             <inertial>
                 <origin xyz="-0.01181 -0.02758 0.0085" rpy="${pi/2} ${pi} -1.903"/>
@@ -590,13 +590,13 @@
                 <material name="Orange"/>
             </collision>
-        </link>
+        </link> -->
         <!-- joint between link_claw2_end and link_claw2_2-->
-        <joint name="${robot_name}_joint_claw1_end_claw2_2" type="fixed">
+        <!-- <joint name="${robot_name}_joint_claw1_end_claw2_2" type="fixed">
             <parent link="${robot_name}_link_claw2_end"/>
             <child link="${robot_name}_link_claw2_2"/>
             <origin xyz="-0.00984 -0.02298 0" rpy="0 0 0"/>
-        </joint>
+        </joint> -->
         <!-- link_claw2_2 -->
-        <link name="${robot_name}_link_claw2_2">
+        <!-- <link name="${robot_name}_link_claw2_2">
             <inertial>
                 <origin xyz="-0.01699 0.01834 0.0135" rpy="${pi/2} ${pi} 2.3057"/>
@@ -619,4 +619,5 @@
             </collision>
         </link>
+ -->
         <xacro:bbot_gazebo robot_name="${robot_name}"/>
         <xacro:bbot_transmission hardware_interface="${hardware_interface}"/>
