Commit message: Updated STL files to meters and updated scaling factor to 1

File: bbot_description/urdf/bbot.xacro (robot description, xacro)
@@ -28,5 +28,5 @@
                 <origin xyz="0 0 0" rpy="${pi/2.0} 0 0"/>
                 <geometry>
-                    <mesh filename="package://bbot_description/meshes/baseplate.stl" scale="0.001 0.001 0.001"/>
+                    <mesh filename="package://bbot_description/meshes/baseplate.stl" scale="1 1 1"/>
                 </geometry>
                 <material name="Orange"/>
@@ -35,5 +35,5 @@
                 <origin xyz="0 0 0" rpy="${pi/2.0} 0 0"/>
                 <geometry>
-                    <mesh filename="package://bbot_description/meshes/baseplate.stl" scale="0.001 0.001 0.001"/>
+                    <mesh filename="package://bbot_description/meshes/baseplate.stl" scale="1 1 1"/>
                 </geometry>
                 <material name="Orange"/>
@@ -54,5 +54,5 @@
                 <origin xyz="0 0 0" rpy="0 0 ${pi/2.0}"/>
                 <geometry>
-                    <mesh filename="package://bbot_description/meshes/motor_no_idler.stl" scale="0.001 0.001 0.001"/>
+                    <mesh filename="package://bbot_description/meshes/motor_no_idler.stl" scale="1 1 1"/>
                 </geometry>
                 <material name="Black"/>
@@ -61,5 +61,5 @@
                 <origin xyz="0 0 0" rpy="0 0 ${pi/2.0}"/>
                 <geometry>
-                    <mesh filename="package://bbot_description/meshes/motor_no_idler.stl" scale="0.001 0.001 0.001"/>
+                    <mesh filename="package://bbot_description/meshes/motor_no_idler.stl" scale="1 1 1"/>
                 </geometry>
                 <material name="Black"/>
@@ -88,5 +88,5 @@
                 <origin xyz="0 0 0" rpy="${pi/2.0} 0 ${pi/2.0}"/>
                 <geometry>
-                    <mesh filename="package://bbot_description/meshes/link1_2.stl" scale="0.001 0.001 0.001"/>
+                    <mesh filename="package://bbot_description/meshes/link1_2.stl" scale="1 1 1"/>
                 </geometry>
                 <material name="Orange"/>
@@ -95,5 +95,5 @@
                 <origin xyz="0 0 0" rpy="${pi/2.0} 0 ${pi/2.0}"/>
                 <geometry>
-                    <mesh filename="package://bbot_description/meshes/link1_2.stl" scale="0.001 0.001 0.001"/>
+                    <mesh filename="package://bbot_description/meshes/link1_2.stl" scale="1 1 1"/>
                 </geometry>
                 <material name="Orange"/>
@@ -114,5 +114,5 @@
                 <origin xyz="0 0 0" rpy="0 0 ${-pi/2.0}"/>
                 <geometry>
-                    <mesh filename="package://bbot_description/meshes/motor_with_idler.stl" scale="0.001 0.001 0.001"/>
+                    <mesh filename="package://bbot_description/meshes/motor_with_idler.stl" scale="1 1 1"/>
                 </geometry>
                 <material name="Black"/>
@@ -121,5 +121,5 @@
                 <origin xyz="0 0 0" rpy="0 0 ${-pi/2.0}"/>
                 <geometry>
-                    <mesh filename="package://bbot_description/meshes/motor_with_idler.stl" scale="0.001 0.001 0.001"/>
+                    <mesh filename="package://bbot_description/meshes/motor_with_idler.stl" scale="1 1 1"/>
                 </geometry>
                 <material name="Black"/>
@@ -148,5 +148,5 @@
                 <origin xyz="0.0275 0 0" rpy="${pi/2.0} ${-pi/2.0} 0"/>
                 <geometry>
-                    <mesh filename="package://bbot_description/meshes/link2_3.stl" scale="0.001 0.001 0.001"/>
+                    <mesh filename="package://bbot_description/meshes/link2_3.stl" scale="1 1 1"/>
                 </geometry>
                 <material name="Orange"/>
@@ -155,5 +155,5 @@
                 <origin xyz="0.0275 0 0" rpy="${pi/2.0} ${-pi/2.0} 0"/>
                 <geometry>
-                    <mesh filename="package://bbot_description/meshes/link2_3.stl" scale="0.001 0.001 0.001"/>
+                    <mesh filename="package://bbot_description/meshes/link2_3.stl" scale="1 1 1"/>
                 </geometry>
                 <material name="Orange"/>
@@ -182,5 +182,5 @@
                 <origin xyz="0 0 0" rpy="0 0 ${pi/2.0}"/>
                 <geometry>
-                    <mesh filename="package://bbot_description/meshes/motor_with_idler.stl" scale="0.001 0.001 0.001"/>
+                    <mesh filename="package://bbot_description/meshes/motor_with_idler.stl" scale="1 1 1"/>
                 </geometry>
                 <material name="Black"/>
@@ -189,5 +189,5 @@
                 <origin xyz="0 0 0" rpy="0 0 ${pi/2.0}"/>
                 <geometry>
-                    <mesh filename="package://bbot_description/meshes/motor_with_idler.stl" scale="0.001 0.001 0.001"/>
+                    <mesh filename="package://bbot_description/meshes/motor_with_idler.stl" scale="1 1 1"/>
                 </geometry>
                 <material name="Black"/>
@@ -208,5 +208,5 @@
                 <origin xyz="0.067 0 0.01" rpy="0 0 0"/>
                 <geometry>
-                    <mesh filename="package://bbot_description/meshes/link3_4.stl" scale="0.001 0.001 0.001"/>
+                    <mesh filename="package://bbot_description/meshes/link3_4.stl" scale="1 1 1"/>
                 </geometry>
                 <material name="Orange"/>
@@ -215,5 +215,5 @@
                 <origin xyz="0.067 0 0.01" rpy="0 0 0"/>
                 <geometry>
-                    <mesh filename="package://bbot_description/meshes/link3_4.stl" scale="0.001 0.001 0.001"/>
+                    <mesh filename="package://bbot_description/meshes/link3_4.stl" scale="1 1 1"/>
                 </geometry>
                 <material name="Orange"/>
@@ -234,5 +234,5 @@
                 <origin xyz="0 0 0" rpy="0 0 ${-pi/2.0}"/>
                 <geometry>
-                    <mesh filename="package://bbot_description/meshes/motor_with_idler.stl" scale="0.001 0.001 0.001"/>
+                    <mesh filename="package://bbot_description/meshes/motor_with_idler.stl" scale="1 1 1"/>
                 </geometry>
                 <material name="Black"/>
@@ -241,5 +241,5 @@
                 <origin xyz="0 0 0" rpy="0 0 ${-pi/2.0}"/>
                 <geometry>
-                    <mesh filename="package://bbot_description/meshes/motor_with_idler.stl" scale="0.001 0.001 0.001"/>
+                    <mesh filename="package://bbot_description/meshes/motor_with_idler.stl" scale="1 1 1"/>
                 </geometry>
                 <material name="Black"/>
@@ -268,5 +268,5 @@
                 <origin xyz="0 0 0.0235" rpy="0 0 0"/>
                 <geometry>
-                    <mesh filename="package://bbot_description/meshes/link4_5.stl" scale="0.001 0.001 0.001"/>
+                    <mesh filename="package://bbot_description/meshes/link4_5.stl" scale="1 1 1"/>
                 </geometry>
                 <material name="Orange"/>
@@ -275,5 +275,5 @@
                 <origin xyz="0 0 0.0235" rpy="0 0 0"/>
                 <geometry>
-                    <mesh filename="package://bbot_description/meshes/link4_5.stl" scale="0.001 0.001 0.001"/>
+                    <mesh filename="package://bbot_description/meshes/link4_5.stl" scale="1 1 1"/>
                 </geometry>
                 <material name="Orange"/>
@@ -302,5 +302,5 @@
                 <origin xyz="0 0 0" rpy="0 0 0"/>
                 <geometry>
-                    <mesh filename="package://bbot_description/meshes/motor_with_idler.stl" scale="0.001 0.001 0.001"/>
+                    <mesh filename="package://bbot_description/meshes/motor_with_idler.stl" scale="1 1 1"/>
                 </geometry>
                 <material name="Black"/>
@@ -309,5 +309,5 @@
                 <origin xyz="0 0 0" rpy="0 0 0"/>
                 <geometry>
-                    <mesh filename="package://bbot_description/meshes/motor_with_idler.stl" scale="0.001 0.001 0.001"/>
+                    <mesh filename="package://bbot_description/meshes/motor_with_idler.stl" scale="1 1 1"/>
                 </geometry>
                 <material name="Black"/>
@@ -328,5 +328,5 @@
                 <origin xyz="0 0 0.0173" rpy="${pi/2.0} 0 ${pi/2.0}"/>
                 <geometry>
-                    <mesh filename="package://bbot_description/meshes/link5_6.stl" scale="0.001 0.001 0.001"/>
+                    <mesh filename="package://bbot_description/meshes/link5_6.stl" scale="1 1 1"/>
                 </geometry>
                 <material name="Orange"/>
@@ -335,5 +335,5 @@
                 <origin xyz="0 0 0.0173" rpy="${pi/2.0} 0 ${pi/2.0}"/>
                 <geometry>
-                    <mesh filename="package://bbot_description/meshes/link5_6.stl" scale="0.001 0.001 0.001"/>
+                    <mesh filename="package://bbot_description/meshes/link5_6.stl" scale="1 1 1"/>
                 </geometry>
                 <material name="Orange"/>
@@ -362,5 +362,5 @@
                 <origin xyz="0 0 0" rpy="0 0 ${pi}"/>
                 <geometry>
-                    <mesh filename="package://bbot_description/meshes/motor_with_idler.stl" scale="0.001 0.001 0.001"/>
+                    <mesh filename="package://bbot_description/meshes/motor_with_idler.stl" scale="1 1 1"/>
                 </geometry>
                 <material name="Black"/>
@@ -369,5 +369,5 @@
                 <origin xyz="0 0 0" rpy="0 0 ${pi}"/>
                 <geometry>
-                    <mesh filename="package://bbot_description/meshes/motor_with_idler.stl" scale="0.001 0.001 0.001"/>
+                    <mesh filename="package://bbot_description/meshes/motor_with_idler.stl" scale="1 1 1"/>
                 </geometry>
                 <material name="Black"/>
@@ -390,5 +390,5 @@
                 <origin xyz="0 0.0175 0.008" rpy="${pi} 0 ${0.0}"/>
                 <geometry>
-                    <mesh filename="package://bbot_description/meshes/gripper_palm.stl" scale="0.001 0.001 0.001"/>
+                    <mesh filename="package://bbot_description/meshes/gripper_palm.stl" scale="1 1 1"/>
                 </geometry>
                 <material name="Orange"/>
@@ -397,5 +397,5 @@
                 <origin xyz="0 0.0175 0.008" rpy="${pi} 0 ${0.0}"/>
                 <geometry>
-                    <mesh filename="package://bbot_description/meshes/gripper_palm.stl" scale="0.001 0.001 0.001"/>
+                    <mesh filename="package://bbot_description/meshes/gripper_palm.stl" scale="1 1 1"/>
                 </geometry>
                 <material name="Orange"/>
@@ -418,5 +418,5 @@
                 <origin xyz="0.015 -0.0115 0.0295" rpy="${pi/2} 0 ${pi}"/>
                 <geometry>
-                    <mesh filename="package://bbot_description/meshes/motor_with_idler.stl" scale="0.001 0.001 0.001"/>
+                    <mesh filename="package://bbot_description/meshes/motor_with_idler.stl" scale="1 1 1"/>
                 </geometry>
                 <material name="Black"/>
@@ -425,5 +425,5 @@
                 <origin xyz="0.015 -0.0115 0.0295" rpy="${pi/2} 0 ${pi}"/>
                 <geometry>
-                    <mesh filename="package://bbot_description/meshes/motor_with_idler.stl" scale="0.001 0.001 0.001"/>
+                    <mesh filename="package://bbot_description/meshes/motor_with_idler.stl" scale="1 1 1"/>
                 </geometry>
                 <material name="Black"/>
@@ -454,5 +454,5 @@
                 <origin xyz="0 0 0" rpy="0 0 ${pi}"/>
                 <geometry>
-                    <mesh filename="package://bbot_description/meshes/gripper_link1_right.stl" scale="0.001 0.001 0.001"/>
+                    <mesh filename="package://bbot_description/meshes/gripper_link1_right.stl" scale="1 1 1"/>
                 </geometry>
                 <material name="Orange"/>
@@ -461,5 +461,5 @@
                 <origin xyz="0 0 0" rpy="0 0 ${pi}"/>
                 <geometry>
-                    <mesh filename="package://bbot_description/meshes/gripper_link1_right.stl" scale="0.001 0.001 0.001"/>
+                    <mesh filename="package://bbot_description/meshes/gripper_link1_right.stl" scale="1 1 1"/>
                 </geometry>
                 <material name="Orange"/>
@@ -495,5 +495,5 @@
                 <origin xyz="-0.01839 -0.01693 0.005" rpy="${-pi/2} 0 -2.3057"/>
                 <geometry>
-                    <mesh filename="package://bbot_description/meshes/gripper_link2.stl" scale="0.001 0.001 0.001"/>
+                    <mesh filename="package://bbot_description/meshes/gripper_link2.stl" scale="1 1 1"/>
                 </geometry>
                 <material name="Orange"/>
@@ -502,5 +502,5 @@
                 <origin xyz="-0.01839 -0.01693 0.005" rpy="${-pi/2} 0 -2.3057"/>
                 <geometry>
-                    <mesh filename="package://bbot_description/meshes/gripper_link2.stl" scale="0.001 0.001 0.001"/>
+                    <mesh filename="package://bbot_description/meshes/gripper_link2.stl" scale="1 1 1"/>
                 </geometry>
                 <material name="Orange"/>
@@ -555,5 +555,5 @@
                 <origin xyz="0.01175 -0.0276 -0.005" rpy="${pi/2} 0 1.903"/>
                 <geometry>
-                    <mesh filename="package://bbot_description/meshes/gripper_link3.stl" scale="0.001 0.001 0.001"/>
+                    <mesh filename="package://bbot_description/meshes/gripper_link3.stl" scale="1 1 1"/>
                 </geometry>
                 <material name="Orange"/>
@@ -562,5 +562,5 @@
                 <origin xyz="0.01175 -0.0276 -0.005" rpy="${pi/2} 0 1.903"/>
                 <geometry>
-                    <mesh filename="package://bbot_description/meshes/gripper_link3.stl" scale="0.001 0.001 0.001"/>
+                    <mesh filename="package://bbot_description/meshes/gripper_link3.stl" scale="1 1 1"/>
                 </geometry>
                 <material name="Orange"/>
@@ -577,5 +577,5 @@
                 <origin xyz="0 0 0.005" rpy="0 ${pi} 3.307"/>
                 <geometry>
-                    <mesh filename="package://bbot_description/meshes/gripper_link1_left.stl" scale="0.001 0.001 0.001"/>
+                    <mesh filename="package://bbot_description/meshes/gripper_link1_left.stl" scale="1 1 1"/>
                 </geometry>
                 <material name="Orange"/>
@@ -584,5 +584,5 @@
                 <origin xyz="0 0 0.005" rpy="0 ${pi} 3.307"/>
                 <geometry>
-                    <mesh filename="package://bbot_description/meshes/gripper_link1_left.stl" scale="0.001 0.001 0.001"/>
+                    <mesh filename="package://bbot_description/meshes/gripper_link1_left.stl" scale="1 1 1"/>
                 </geometry>
                 <material name="Orange"/>
@@ -618,5 +618,5 @@
                 <origin xyz="0.01699 -0.01834 0.005" rpy="${pi/2} ${pi} 2.3057"/>
                 <geometry>
-                    <mesh filename="package://bbot_description/meshes/gripper_link2.stl" scale="0.001 0.001 0.001"/>
+                    <mesh filename="package://bbot_description/meshes/gripper_link2.stl" scale="1 1 1"/>
                 </geometry>
                 <material name="Orange"/>
@@ -625,5 +625,5 @@
                 <origin xyz="0.01699 -0.01834 0.005" rpy="${pi/2} ${pi} 2.3057"/>
                 <geometry>
-                    <mesh filename="package://bbot_description/meshes/gripper_link2.stl" scale="0.001 0.001 0.001"/>
+                    <mesh filename="package://bbot_description/meshes/gripper_link2.stl" scale="1 1 1"/>
                 </geometry>
                 <material name="Orange"/>
@@ -631,5 +631,5 @@
         </link>
         <!-- joint between link_claw2 and link_claw2_end-->
-        <joint name="${robot_name}_joint_claw2_claw2_end" type="continuous">
+        <joint name="${robot_name}_joint_claw2_claw2_end" type="revolute">
             <parent link="${robot_name}_link_claw2"/>
             <child link="${robot_name}_link_claw2_end"/>
@@ -659,5 +659,5 @@
                 <origin xyz="-0.01181 -0.02758 0" rpy="${pi/2} ${pi} -1.903"/>
                 <geometry>
-                    <mesh filename="package://bbot_description/meshes/gripper_link3.stl" scale="0.001 0.001 0.001"/>
+                    <mesh filename="package://bbot_description/meshes/gripper_link3.stl" scale="1 1 1"/>
                 </geometry>
                 <material name="Orange"/>
@@ -666,5 +666,5 @@
                 <origin xyz="-0.01181 -0.02758 0" rpy="${pi/2} ${pi} -1.903"/>
                 <geometry>
-                    <mesh filename="package://bbot_description/meshes/gripper_link3.stl" scale="0.001 0.001 0.001"/>
+                    <mesh filename="package://bbot_description/meshes/gripper_link3.stl" scale="1 1 1"/>
                 </geometry>
                 <material name="Orange"/>

Commit message: Added aruco markers to cups and aruco holder to base

File: bbot_description/urdf/bbot.xacro (robot description, xacro)
@@ -673,4 +673,29 @@
         <xacro:bbot_gazebo robot_name="${robot_name}"/>
         <xacro:bbot_transmission hardware_interface="${hardware_interface}"/>
+        <!-- Aruco marker joints and links -->
+        <joint name="${robot_name}_joint_baseplate_arucobase" type="fixed">
+            <parent link="${robot_name}_link_baseplate"/>
+            <child link="${robot_name}_link_arucobase"/>
+            <origin xyz="0.08241 0 0" rpy="${pi/2.0} 0 ${-pi/2.0}"/>
+        </joint>
+        <link name="${robot_name}_link_arucobase">
+            <inertial>
+                <origin xyz="0 0 0" rpy="0 0 0"/>
+                <mass value="0.006"/>
+                <inertia ixx="0" ixy="0" ixz="0" iyy="0.000003" iyz="0" izz="0.000003"/>
+            </inertial>
+            <visual>
+                <origin xyz="0 0 0" rpy="0 0 0"/>
+                <geometry>
+                    <mesh filename="package://bbot_description/meshes/aruco_holder.stl"/>
+                </geometry>
+            </visual>
+            <collision>
+                <origin xyz="0 0 0" rpy="0 0 0"/>
+                <geometry>
+                    <mesh filename="package://bbot_description/meshes/aruco_holder.stl"/>
+                </geometry>
+            </collision>
+        </link>
     </xacro:macro>
 </robot>

File: bbot_description/urdf/ingredient_cup.xacro (robot description, xacro)
@@ -78,5 +78,5 @@
 				<origin xyz="0.0 0 0" rpy="0.0 0 0"/>
 				<geometry>
-					<mesh filename="package://bbot_aruco/markers/aruco_99_50mm.dae"/>
+					<mesh filename="package://${aruco_dae_path}"/>
 				</geometry>
 			</collision>
@@ -84,5 +84,5 @@
 				<origin rpy="0.0 0 0" xyz="0.0 0 0"/>
 				<geometry>
-					<mesh filename="package://bbot_aruco/markers/aruco_99_50mm.dae"/>
+					<mesh filename="package://${aruco_dae_path}"/>
 				</geometry>
 			</visual>

Commit message: Added camera to the Gazebo scene

File: bbot_description/urdf/bbot.xacro (robot description, xacro)
@@ -698,4 +698,28 @@
             </collision>
         </link>
+        <joint name="${robot_name}_joint_arucobase_aruco" type="fixed">
+            <parent link="${robot_name}_link_arucobase"/>
+            <child link="${robot_name}_link_arucorobot"/>
+            <origin xyz="0 0.026 0.0005" rpy="0 ${pi} ${pi}"/>
+        </joint>
+        <link name="${robot_name}_link_arucorobot">
+            <inertial>
+                <origin xyz="0 0 0" rpy="0 0 0"/>
+                <mass value="0.006"/>
+                <inertia ixx="0" ixy="0" ixz="0" iyy="0.000003" iyz="0" izz="0.000003"/>
+            </inertial>
+            <visual>
+                <origin xyz="0 0 0" rpy="0 0 0"/>
+                <geometry>
+                    <mesh filename="package://bbot_aruco/markers/aruco_26_50mm.dae"/>
+                </geometry>
+            </visual>
+            <collision>
+                <origin xyz="0 0 0" rpy="0 0 0"/>
+                <geometry>
+                    <mesh filename="package://bbot_aruco/markers/aruco_26_50mm.dae"/>
+                </geometry>
+            </collision>
+        </link>
     </xacro:macro>
 </robot>

Commit message: Update IK to account for EE offset, modified damping in bbot.xacro, tuned some pose gains

File: bbot_description/urdf/bbot.xacro (robot description, xacro)
@@ -9,5 +9,5 @@
     <xacro:property name="safety_controller_k_pos" value="100" />
     <xacro:property name="safety_controller_k_vel" value="2" />
-    <xacro:property name="joint_damping" value="0.5" />
+    <xacro:property name="joint_damping" value="0.01" />
     <xacro:property name="max_effort" value="300"/>
     <xacro:property name="max_velocity" value="10"/>
@@ -380,5 +380,5 @@
             <origin xyz="0 0 0.015" rpy="0 0 0"/>
         </joint>
-       <!-- link gripper_palm -->
+        <!-- link gripper_palm -->
         <link name="${robot_name}_gripper_palm">
             <inertial>
