Commit message: Finished updating state machine with static transformations

File: bbot_description/urdf/bbot.xacro (robot description, xacro)
@@ -9,7 +9,8 @@
     <xacro:property name="safety_controller_k_pos" value="100" />
     <xacro:property name="safety_controller_k_vel" value="2" />
-    <xacro:property name="joint_damping" value="0.5" />
+    <xacro:property name="joint_damping" value="0.01" />
     <xacro:property name="max_effort" value="300"/>
     <xacro:property name="max_velocity" value="10"/>
+    <xacro:property name="scaling" value="100"/>
     <xacro:macro name="bbot" params="parent hardware_interface robot_name *origin">
         <!-- joint between parent (a.k.a. world) and link_0 -->
@@ -23,5 +24,5 @@
                 <origin xyz="0 0 0" rpy="${pi/2.0} 0 0"/>
                 <mass value="0.0800"/>
-                <inertia ixx="0.000070" ixy="0" ixz="0" iyy="0.000174" iyz="0" izz="0.000107"/>
+                <inertia ixx="${scaling*0.000069}" ixy="0" ixz="0" iyy="${scaling*0.000174}" iyz="0" izz="${scaling*0.000106}"/>
             </inertial>
             <visual>
@@ -49,5 +50,5 @@
                 <origin xyz="0 0 0" rpy="0 0 ${pi/2.0}"/>
                 <mass value="0.074"/>
-                <inertia ixx="0.000031" ixy="0" ixz="0" iyy="0.000013" iyz="0" izz="0.000027"/>
+                <inertia ixx="${scaling*0.000021}" ixy="0" ixz="0" iyy="${scaling*0.000013}" iyz="${scaling*0.000001}" izz="${scaling*0.000018}"/>
             </inertial>
             <visual>
@@ -83,5 +84,5 @@
                 <origin xyz="0 0 0" rpy="${pi/2.0} 0 ${pi/2.0}"/>
                 <mass value="0.0296"/>
-                <inertia ixx="0.000028" ixy="0" ixz="0" iyy="0.000014" iyz="0" izz="0.000023"/>
+                <inertia ixx="${scaling*0.000017}" ixy="0" ixz="0" iyy="${scaling*0.000014}" iyz="0" izz="${scaling*0.000012}"/>
             </inertial>
             <visual>
@@ -109,5 +110,5 @@
                 <origin xyz="0 0 0" rpy="0 0 ${-pi/2.0}"/>
                 <mass value="0.076"/>
-                <inertia ixx="0.000031" ixy="0" ixz="0" iyy="0.000014" iyz="0" izz="0.000027"/>
+                <inertia ixx="${scaling*0.000022}" ixy="0" ixz="0" iyy="${scaling*0.000014}" iyz="0" izz="${scaling*0.000018}"/>
             </inertial>
             <visual>
@@ -143,5 +144,5 @@
                 <origin xyz="0.0275 0 0" rpy="${pi/2.0} ${-pi/2.0} 0"/>
                 <mass value="0.0584"/>
-                <inertia ixx="0.000096" ixy="0" ixz="0" iyy="0.000021" iyz="0" izz="0.00011"/>
+                <inertia ixx="${scaling*0.000059}" ixy="0" ixz="0" iyy="${scaling*0.000021}" iyz="0" izz="${scaling*0.000074}"/>
             </inertial>
             <visual>
@@ -177,5 +178,5 @@
                 <origin xyz="0 0 0" rpy="0 0 ${pi/2.0}"/>
                 <mass value="0.076"/>
-                <inertia ixx="0.000031" ixy="0" ixz="0" iyy="0.000014" iyz="0" izz="0.000027"/>
+                <inertia ixx="${scaling*0.000022}" ixy="0" ixz="0" iyy="${scaling*0.000014}" iyz="0" izz="${scaling*0.000018}"/>
             </inertial>
             <visual>
@@ -203,5 +204,5 @@
                 <origin xyz="0.067 0 0.01" rpy="0 0 0"/>
                 <mass value="0.0409"/>
-                <inertia ixx="0.0027" ixy="-0.0001" ixz="0" iyy="0" iyz="0" izz="0.0027"/>
+                <inertia ixx="${scaling*0.0027}" ixy="${scaling*-0.0001}" ixz="0" iyy="0" iyz="0" izz="${scaling*0.0027}"/>
             </inertial>
             <visual>
@@ -229,5 +230,5 @@
                 <origin xyz="0 0 0" rpy="0 0 ${-pi/2.0}"/>
                 <mass value="0.076"/>
-                <inertia ixx="0.000031" ixy="0" ixz="0" iyy="0.000014" iyz="0" izz="0.000027"/>
+                <inertia ixx="${scaling*0.000022}" ixy="0" ixz="0" iyy="${scaling*0.000014}" iyz="0" izz="${scaling*0.000018}"/>
             </inertial>
             <visual>
@@ -263,5 +264,5 @@
                 <origin xyz="0 0 0.0235" rpy="0 0 0"/>
                 <mass value="0.021"/>
-                <inertia ixx="0.000016" ixy="0" ixz="0" iyy="0.000008" iyz="0" izz="0.00001"/>
+                <inertia ixx="${scaling*0.000013}" ixy="0" ixz="0" iyy="${scaling*0.000005}" iyz="0" izz="${scaling*0.00001}"/>
             </inertial>
             <visual>
@@ -297,5 +298,5 @@
                 <origin xyz="0 0 0" rpy="0 0 0"/>
                 <mass value="0.076"/>
-                <inertia ixx="0.000031" ixy="0" ixz="0" iyy="0.000014" iyz="0" izz="0.000027"/>
+                <inertia ixx="${scaling*0.000022}" ixy="0" ixz="0" iyy="${scaling*0.000014}" iyz="0" izz="${scaling*0.000018}"/>
             </inertial>
             <visual>
@@ -323,5 +324,5 @@
                 <origin xyz="0 0 0.0173" rpy="${pi/2.0} 0 ${pi/2.0}"/>
                 <mass value="0.01588"/>
-                <inertia ixx="0.00001" ixy="0.000002" ixz="0" iyy="0.000003" iyz="0" izz="0.000009"/>
+                <inertia ixx="${scaling*0.000005}" ixy="0" ixz="0" iyy="${scaling*0.000003}" iyz="0" izz="${scaling*0.000004}"/>
             </inertial>
             <visual>
@@ -357,5 +358,5 @@
                 <origin xyz="0 0 0" rpy="0 0 ${pi}"/>
                 <mass value="0.076"/>
-                <inertia ixx="0.000031" ixy="0" ixz="0" iyy="0.000014" iyz="0" izz="0.000027"/>
+                <inertia ixx="${scaling*0.000021}" ixy="0" ixz="0" iyy="${scaling*0.000013}" iyz="0" izz="${scaling*0.000018}"/>
             </inertial>
             <visual>
@@ -385,5 +386,5 @@
                 <origin xyz="0 0.0175 0.008" rpy="${pi} 0 ${0.0}"/>
                 <mass value="0.07825"/>
-                <inertia ixx="0.00013" ixy="-0.000001" ixz="0" iyy="0.000141" iyz="-0.000015" izz="0.00003"/>
+                <inertia ixx="${scaling*0.000068}" ixy="0" ixz="${scaling*-0.000001}" iyy="${scaling*0.000082}" iyz="${scaling*-0.000001}" izz="${scaling*0.000027}"/>
             </inertial>
             <visual>
@@ -413,5 +414,5 @@
                 <origin xyz="0.015 -0.0115 0.0295" rpy="${pi/2} 0 ${pi}"/>
                 <mass value="0.076"/>
-                <inertia ixx="0.000031" ixy="0" ixz="0" iyy="0.000014" iyz="0" izz="0.000027"/>
+                <inertia ixx="${scaling*0.000022}" ixy="0" ixz="0" iyy="${scaling*0.000014}" iyz="0" izz="${scaling*0.000018}"/>
             </inertial>
             <visual>
@@ -449,5 +450,5 @@
                 <origin xyz="0 0 0" rpy="0 0 ${pi}"/>
                 <mass value="0.0065"/>
-                <inertia ixx="0.000003" ixy="0.000003" ixz="0" iyy="0.000003" iyz="0" izz="0.000006"/>
+                <inertia ixx="${scaling*0.000001}" ixy="${scaling*0.000001}" ixz="0" iyy="${scaling*0.000002}" iyz="0" izz="${scaling*0.000003}"/>
             </inertial>
             <visual>
@@ -490,5 +491,5 @@
                 <origin xyz="-0.01839 -0.01693 0.005" rpy="${-pi/2} 0 -2.3057"/>
                 <mass value=".00455"/>
-                <inertia ixx="0" ixy="0" ixz="0" iyy="0.000001" iyz="0" izz="0.000001"/>
+                <inertia ixx="${scaling*0.0000001}" ixy="0" ixz="0" iyy="${scaling*0.000001}" iyz="0" izz="${scaling*0.000001}"/>
             </inertial>
             <visual>
@@ -550,5 +551,5 @@
                 <origin xyz="0.01175 -0.0276 -0.005" rpy="${pi/2} 0 1.903"/>
                 <mass value="0.006"/>
-                <inertia ixx="0" ixy="0" ixz="0" iyy="0.000003" iyz="0" izz="0.000003"/>
+                <inertia ixx="${scaling*0.0000001}" ixy="0" ixz="0" iyy="${scaling*0.000003}" iyz="0" izz="${scaling*0.000003}"/>
             </inertial>
             <visual>
@@ -572,5 +573,5 @@
                 <origin xyz="0 0 0.005" rpy="0 ${pi} 3.307"/>
                 <mass value=".0066"/>
-                <inertia ixx="0.000004" ixy="0.000003" ixz="0" iyy="0.000002" iyz="0.000001" izz="0.000006"/>
+                <inertia ixx="${scaling*0.000002}" ixy="${scaling*0.000001}" ixz="0" iyy="${scaling*0.000001}" iyz="0" izz="${scaling*0.000003}"/>
             </inertial>
             <visual>
@@ -613,5 +614,5 @@
                 <origin xyz="0.01699 -0.01834 0.005" rpy="${pi/2} ${pi} 2.3057"/>
                 <mass value=".00455"/>
-                <inertia ixx="0" ixy="0" ixz="0" iyy="0.000001" iyz="0" izz="0.000001"/>
+                <inertia ixx="${scaling*0.0000001}" ixy="0" ixz="0" iyy="${scaling*0.000001}" iyz="0" izz="${scaling*0.000001}"/>
             </inertial>
             <visual>
@@ -654,5 +655,5 @@
                 <origin xyz="-0.01181 -0.02758 0" rpy="${pi/2} ${pi} -1.903"/>
                 <mass value="0.006"/>
-                <inertia ixx="0" ixy="0" ixz="0" iyy="0.000003" iyz="0" izz="0.000003"/>
+                <inertia ixx="${scaling*0.0000001}" ixy="0" ixz="0" iyy="${scaling*0.000003}" iyz="0" izz="${scaling*0.000003}"/>
             </inertial>
             <visual>

File: bbot_description/urdf/bbot_camera.gazebo.xacro (robot description, xacro)
@@ -10,5 +10,5 @@
     <gazebo reference="bbot_camera_link">
       <sensor type="camera" name="camera1">
-        <update_rate>30.0</update_rate>
+        <update_rate>10.0</update_rate>
         <camera name="head">
           <horizontal_fov>1.3962634</horizontal_fov>

Commit message: Updated IK to account for world to zero frame translation, tuned joint 1 gains

File: bbot_description/urdf/bbot.xacro (robot description, xacro)
@@ -12,4 +12,5 @@
     <xacro:property name="max_effort" value="300"/>
     <xacro:property name="max_velocity" value="10"/>
+    <xacro:property name="scaling" value="100"/>
     <xacro:macro name="bbot" params="parent hardware_interface robot_name *origin">
         <!-- joint between parent (a.k.a. world) and link_0 -->
@@ -23,5 +24,5 @@
                 <origin xyz="0 0 0" rpy="${pi/2.0} 0 0"/>
                 <mass value="0.0800"/>
-                <inertia ixx="0.000070" ixy="0" ixz="0" iyy="0.000174" iyz="0" izz="0.000107"/>
+                <inertia ixx="${scaling*0.000069}" ixy="0" ixz="0" iyy="${scaling*0.000174}" iyz="0" izz="${scaling*0.000106}"/>
             </inertial>
             <visual>
@@ -49,5 +50,5 @@
                 <origin xyz="0 0 0" rpy="0 0 ${pi/2.0}"/>
                 <mass value="0.074"/>
-                <inertia ixx="0.000031" ixy="0" ixz="0" iyy="0.000013" iyz="0" izz="0.000027"/>
+                <inertia ixx="${scaling*0.000021}" ixy="0" ixz="0" iyy="${scaling*0.000013}" iyz="${scaling*0.000001}" izz="${scaling*0.000018}"/>
             </inertial>
             <visual>
@@ -83,5 +84,5 @@
                 <origin xyz="0 0 0" rpy="${pi/2.0} 0 ${pi/2.0}"/>
                 <mass value="0.0296"/>
-                <inertia ixx="0.000028" ixy="0" ixz="0" iyy="0.000014" iyz="0" izz="0.000023"/>
+                <inertia ixx="${scaling*0.000017}" ixy="0" ixz="0" iyy="${scaling*0.000014}" iyz="0" izz="${scaling*0.000012}"/>
             </inertial>
             <visual>
@@ -109,5 +110,5 @@
                 <origin xyz="0 0 0" rpy="0 0 ${-pi/2.0}"/>
                 <mass value="0.076"/>
-                <inertia ixx="0.000031" ixy="0" ixz="0" iyy="0.000014" iyz="0" izz="0.000027"/>
+                <inertia ixx="${scaling*0.000022}" ixy="0" ixz="0" iyy="${scaling*0.000014}" iyz="0" izz="${scaling*0.000018}"/>
             </inertial>
             <visual>
@@ -143,5 +144,5 @@
                 <origin xyz="0.0275 0 0" rpy="${pi/2.0} ${-pi/2.0} 0"/>
                 <mass value="0.0584"/>
-                <inertia ixx="0.000096" ixy="0" ixz="0" iyy="0.000021" iyz="0" izz="0.00011"/>
+                <inertia ixx="${scaling*0.000059}" ixy="0" ixz="0" iyy="${scaling*0.000021}" iyz="0" izz="${scaling*0.000074}"/>
             </inertial>
             <visual>
@@ -177,5 +178,5 @@
                 <origin xyz="0 0 0" rpy="0 0 ${pi/2.0}"/>
                 <mass value="0.076"/>
-                <inertia ixx="0.000031" ixy="0" ixz="0" iyy="0.000014" iyz="0" izz="0.000027"/>
+                <inertia ixx="${scaling*0.000022}" ixy="0" ixz="0" iyy="${scaling*0.000014}" iyz="0" izz="${scaling*0.000018}"/>
             </inertial>
             <visual>
@@ -203,5 +204,5 @@
                 <origin xyz="0.067 0 0.01" rpy="0 0 0"/>
                 <mass value="0.0409"/>
-                <inertia ixx="0.0027" ixy="-0.0001" ixz="0" iyy="0" iyz="0" izz="0.0027"/>
+                <inertia ixx="${scaling*0.0027}" ixy="${scaling*-0.0001}" ixz="0" iyy="0" iyz="0" izz="${scaling*0.0027}"/>
             </inertial>
             <visual>
@@ -229,5 +230,5 @@
                 <origin xyz="0 0 0" rpy="0 0 ${-pi/2.0}"/>
                 <mass value="0.076"/>
-                <inertia ixx="0.000031" ixy="0" ixz="0" iyy="0.000014" iyz="0" izz="0.000027"/>
+                <inertia ixx="${scaling*0.000022}" ixy="0" ixz="0" iyy="${scaling*0.000014}" iyz="0" izz="${scaling*0.000018}"/>
             </inertial>
             <visual>
@@ -263,5 +264,5 @@
                 <origin xyz="0 0 0.0235" rpy="0 0 0"/>
                 <mass value="0.021"/>
-                <inertia ixx="0.000016" ixy="0" ixz="0" iyy="0.000008" iyz="0" izz="0.00001"/>
+                <inertia ixx="${scaling*0.000013}" ixy="0" ixz="0" iyy="${scaling*0.000005}" iyz="0" izz="${scaling*0.00001}"/>
             </inertial>
             <visual>
@@ -297,5 +298,5 @@
                 <origin xyz="0 0 0" rpy="0 0 0"/>
                 <mass value="0.076"/>
-                <inertia ixx="0.000031" ixy="0" ixz="0" iyy="0.000014" iyz="0" izz="0.000027"/>
+                <inertia ixx="${scaling*0.000022}" ixy="0" ixz="0" iyy="${scaling*0.000014}" iyz="0" izz="${scaling*0.000018}"/>
             </inertial>
             <visual>
@@ -323,5 +324,5 @@
                 <origin xyz="0 0 0.0173" rpy="${pi/2.0} 0 ${pi/2.0}"/>
                 <mass value="0.01588"/>
-                <inertia ixx="0.00001" ixy="0.000002" ixz="0" iyy="0.000003" iyz="0" izz="0.000009"/>
+                <inertia ixx="${scaling*0.000005}" ixy="0" ixz="0" iyy="${scaling*0.000003}" iyz="0" izz="${scaling*0.000004}"/>
             </inertial>
             <visual>
@@ -357,5 +358,5 @@
                 <origin xyz="0 0 0" rpy="0 0 ${pi}"/>
                 <mass value="0.076"/>
-                <inertia ixx="0.000031" ixy="0" ixz="0" iyy="0.000014" iyz="0" izz="0.000027"/>
+                <inertia ixx="${scaling*0.000021}" ixy="0" ixz="0" iyy="${scaling*0.000013}" iyz="0" izz="${scaling*0.000018}"/>
             </inertial>
             <visual>
@@ -380,10 +381,10 @@
             <origin xyz="0 0 0.015" rpy="0 0 0"/>
         </joint>
-        <!-- link gripper_palm -->
+       <!-- link gripper_palm -->
         <link name="${robot_name}_gripper_palm">
             <inertial>
                 <origin xyz="0 0.0175 0.008" rpy="${pi} 0 ${0.0}"/>
                 <mass value="0.07825"/>
-                <inertia ixx="0.00013" ixy="-0.000001" ixz="0" iyy="0.000141" iyz="-0.000015" izz="0.00003"/>
+                <inertia ixx="${scaling*0.000068}" ixy="0" ixz="${scaling*-0.000001}" iyy="${scaling*0.000082}" iyz="${scaling*-0.000001}" izz="${scaling*0.000027}"/>
             </inertial>
             <visual>
@@ -413,5 +414,5 @@
                 <origin xyz="0.015 -0.0115 0.0295" rpy="${pi/2} 0 ${pi}"/>
                 <mass value="0.076"/>
-                <inertia ixx="0.000031" ixy="0" ixz="0" iyy="0.000014" iyz="0" izz="0.000027"/>
+                <inertia ixx="${scaling*0.000022}" ixy="0" ixz="0" iyy="${scaling*0.000014}" iyz="0" izz="${scaling*0.000018}"/>
             </inertial>
             <visual>
@@ -449,5 +450,5 @@
                 <origin xyz="0 0 0" rpy="0 0 ${pi}"/>
                 <mass value="0.0065"/>
-                <inertia ixx="0.000003" ixy="0.000003" ixz="0" iyy="0.000003" iyz="0" izz="0.000006"/>
+                <inertia ixx="${scaling*0.000001}" ixy="${scaling*0.000001}" ixz="0" iyy="${scaling*0.000002}" iyz="0" izz="${scaling*0.000003}"/>
             </inertial>
             <visual>
@@ -490,5 +491,5 @@
                 <origin xyz="-0.01839 -0.01693 0.005" rpy="${-pi/2} 0 -2.3057"/>
                 <mass value=".00455"/>
-                <inertia ixx="0" ixy="0" ixz="0" iyy="0.000001" iyz="0" izz="0.000001"/>
+                <inertia ixx="${scaling*0.0000001}" ixy="0" ixz="0" iyy="${scaling*0.000001}" iyz="0" izz="${scaling*0.000001}"/>
             </inertial>
             <visual>
@@ -550,5 +551,5 @@
                 <origin xyz="0.01175 -0.0276 -0.005" rpy="${pi/2} 0 1.903"/>
                 <mass value="0.006"/>
-                <inertia ixx="0" ixy="0" ixz="0" iyy="0.000003" iyz="0" izz="0.000003"/>
+                <inertia ixx="${scaling*0.0000001}" ixy="0" ixz="0" iyy="${scaling*0.000003}" iyz="0" izz="${scaling*0.000003}"/>
             </inertial>
             <visual>
@@ -572,5 +573,5 @@
                 <origin xyz="0 0 0.005" rpy="0 ${pi} 3.307"/>
                 <mass value=".0066"/>
-                <inertia ixx="0.000004" ixy="0.000003" ixz="0" iyy="0.000002" iyz="0.000001" izz="0.000006"/>
+                <inertia ixx="${scaling*0.000002}" ixy="${scaling*0.000001}" ixz="0" iyy="${scaling*0.000001}" iyz="0" izz="${scaling*0.000003}"/>
             </inertial>
             <visual>
@@ -613,5 +614,5 @@
                 <origin xyz="0.01699 -0.01834 0.005" rpy="${pi/2} ${pi} 2.3057"/>
                 <mass value=".00455"/>
-                <inertia ixx="0" ixy="0" ixz="0" iyy="0.000001" iyz="0" izz="0.000001"/>
+                <inertia ixx="${scaling*0.0000001}" ixy="0" ixz="0" iyy="${scaling*0.000001}" iyz="0" izz="${scaling*0.000001}"/>
             </inertial>
             <visual>
@@ -654,5 +655,5 @@
                 <origin xyz="-0.01181 -0.02758 0" rpy="${pi/2} ${pi} -1.903"/>
                 <mass value="0.006"/>
-                <inertia ixx="0" ixy="0" ixz="0" iyy="0.000003" iyz="0" izz="0.000003"/>
+                <inertia ixx="${scaling*0.0000001}" ixy="0" ixz="0" iyy="${scaling*0.000003}" iyz="0" izz="${scaling*0.000003}"/>
             </inertial>
             <visual>
