Commit message: Fixed gripper mimic joints

File: bbot_description/urdf/bbot.xacro (robot description, xacro)
@@ -407,51 +407,49 @@
             <parent link="${robot_name}_gripper_palm"/>
             <child link="${robot_name}_link_motor7"/>
-            <origin xyz="-0.0305 -0.0065 0.0215" rpy="0 0 0"/>
+            <origin xyz="-0.0155 -0.018 0.0513" rpy="0 0 0"/>
         </joint>
         <!-- motor 7 -->
         <link name="${robot_name}_link_motor7">
             <inertial>
-                <origin xyz="0.015 -0.0115 0.0295" rpy="${pi/2} 0 ${pi}"/>
+                <origin xyz="0 0 0" rpy="${pi/2} 0 ${pi}"/>
                 <mass value="0.076"/>
                 <inertia ixx="${scaling*0.000022}" ixy="0" ixz="0" iyy="${scaling*0.000014}" iyz="0" izz="${scaling*0.000018}"/>
             </inertial>
             <visual>
-                <origin xyz="0.015 -0.0115 0.0295" rpy="${pi/2} 0 ${pi}"/>
-                <geometry>
-                    <mesh filename="package://bbot_description/meshes/motor_with_idler.stl" scale="1 1 1"/>
-                </geometry>
-                <material name="Black"/>
-            </visual>
-            <collision>
-                <origin xyz="0.015 -0.0115 0.0295" rpy="${pi/2} 0 ${pi}"/>
-                <geometry>
-                    <mesh filename="package://bbot_description/meshes/motor_with_idler.stl" scale="1 1 1"/>
-                </geometry>
-                <material name="Black"/>
-            </collision>
-        </link>
-        <!-- joint between motor 7 and link_claw1-->
+                <origin xyz="0 0 0" rpy="${pi/2} 0 ${pi}"/>
+                <geometry>
+                    <mesh filename="package://bbot_description/meshes/motor_with_idler.stl" scale="1 1 1"/>
+                </geometry>
+                <material name="Black"/>
+            </visual>
+            <collision>
+                <origin xyz="0 0 0" rpy="${pi/2} 0 ${pi}"/>
+                <geometry>
+                    <mesh filename="package://bbot_description/meshes/motor_with_idler.stl" scale="1 1 1"/>
+                </geometry>
+                <material name="Black"/>
+            </collision>
+        </link>
         <joint name="${robot_name}_joint_7" type="revolute">
             <parent link="${robot_name}_link_motor7"/>
             <child link="${robot_name}_link_claw1"/>
-            <origin xyz="0.015 0.009 0.0295" rpy="${-pi/2} 0 0"/>
-            <axis xyz="0 0 1"/>
-            <limit lower="${-170 * pi / 180}" upper="${170 * pi / 180}"
-                effort="${max_effort}" velocity="${max_velocity}" />
-            <safety_controller soft_lower_limit="${-168 * pi / 180}"
-                     soft_upper_limit="${168 * pi / 180}"
-                     k_position="${safety_controller_k_pos}"
-                     k_velocity="${safety_controller_k_vel}"/>
-            <dynamics damping="${joint_damping}"/>
-        </joint>
-        <!-- link_claw1 -->
+            <origin xyz="0 0 0" rpy="${-pi/2} 0 0"/>
+            <axis xyz="0 0 1"/>
+            <limit lower="${-170 * pi / 180}" upper="${170 * pi / 180}"
+                effort="${max_effort}" velocity="${max_velocity}" />
+            <safety_controller soft_lower_limit="${-168 * pi / 180}"
+                     soft_upper_limit="${168 * pi / 180}"
+                     k_position="${safety_controller_k_pos}"
+                     k_velocity="${safety_controller_k_vel}"/>
+            <dynamics damping="${joint_damping}"/>
+        </joint>
         <link name="${robot_name}_link_claw1">
             <inertial>
-                <origin xyz="0 0 0" rpy="0 0 ${pi}"/>
+                <origin xyz="0 0 0.0205" rpy="0 0 ${pi}"/>
                 <mass value="0.0065"/>
                 <inertia ixx="${scaling*0.000001}" ixy="${scaling*0.000001}" ixz="0" iyy="${scaling*0.000002}" iyz="0" izz="${scaling*0.000003}"/>
             </inertial>
             <visual>
-                <origin xyz="0 0 0" rpy="0 0 ${pi}"/>
+                <origin xyz="0 0 0.0205" rpy="0 0 ${pi}"/>
                 <geometry>
                     <mesh filename="package://bbot_description/meshes/gripper_link1_right.stl" scale="1 1 1"/>
@@ -460,5 +458,5 @@
             </visual>
             <collision>
-                <origin xyz="0 0 0" rpy="0 0 ${pi}"/>
+                <origin xyz="0 0 0.0205" rpy="0 0 ${pi}"/>
                 <geometry>
                     <mesh filename="package://bbot_description/meshes/gripper_link1_right.stl" scale="1 1 1"/>
@@ -467,9 +465,8 @@
             </collision>
         </link>
-        <!-- joint between link_claw1 and link_claw1_2-->
         <joint name="${robot_name}_joint_claw1_claw1_2" type="revolute">
-            <parent link="${robot_name}_link_claw1"/>
+            <parent link="${robot_name}_link_motor7"/>
             <child link="${robot_name}_link_claw1_2"/>
-            <origin xyz="0.008 -0.024 0" rpy="0 0 0"/>
+            <origin xyz="0.008 0.0205 0.024" rpy="${-pi/2} 0 0"/>
             <axis xyz="0 0 1"/>
             <limit lower="${-170 * pi / 180}" upper="${170 * pi / 180}"
@@ -486,5 +483,4 @@
             mimic_joint="${robot_name}_joint_claw1_claw1_2"
             has_pid="false" multiplier="1.0" max_effort="${max_effort}" />
-        <!-- link_claw1_2 -->
         <link name="${robot_name}_link_claw1_2">
             <inertial>
@@ -508,9 +504,47 @@
             </collision>
         </link>
-        <!-- joint between link_claw1 and link_claw2-->
+        <joint name="${robot_name}_joint_claw1_claw1_end" type="revolute">
+            <parent link="${robot_name}_link_claw1"/>
+            <child link="${robot_name}_link_claw1_end"/>
+            <origin xyz="-0.03858 -0.03858 0.0205" rpy="0 0 0"/>
+            <axis xyz="0 0 1"/>
+            <limit lower="${-170 * pi / 180}" upper="${170 * pi / 180}"
+                effort="${max_effort}" velocity="${max_velocity}" />
+            <safety_controller soft_lower_limit="${-168 * pi / 180}"
+                     soft_upper_limit="${168 * pi / 180}"
+                     k_position="${safety_controller_k_pos}"
+                     k_velocity="${safety_controller_k_vel}"/>
+            <dynamics damping="${joint_damping}"/>
+            <mimic joint="${robot_name}_joint_7" multiplier="-1.0" offset = "0"/>
+        </joint>
+        <xacro:mimic_joint_plugin_gazebo name_prefix="${robot_name}_joint_claw1_claw1_end"
+            parent_joint="${robot_name}_joint_7"
+            mimic_joint="${robot_name}_joint_claw1_claw1_end"
+            has_pid="false" multiplier="-1.0" max_effort="${max_effort}" />
+        <link name="${robot_name}_link_claw1_end">
+            <inertial>
+                <origin xyz="0.01175 -0.0276 -0.005" rpy="${pi/2} 0 1.903"/>
+                <mass value="0.006"/>
+                <inertia ixx="${scaling*0.0000001}" ixy="0" ixz="0" iyy="${scaling*0.000003}" iyz="0" izz="${scaling*0.000003}"/>
+            </inertial>
+            <visual>
+                <origin xyz="0.01175 -0.0276 -0.005" rpy="${pi/2} 0 1.903"/>
+                <geometry>
+                    <mesh filename="package://bbot_description/meshes/gripper_link3.stl" scale="1 1 1"/>
+                </geometry>
+                <material name="Orange"/>
+            </visual>
+            <collision>
+                <origin xyz="0.01175 -0.0276 -0.005" rpy="${pi/2} 0 1.903"/>
+                <geometry>
+                    <mesh filename="package://bbot_description/meshes/gripper_link3.stl" scale="1 1 1"/>
+                </geometry>
+                <material name="Orange"/>
+            </collision>
+        </link>
         <joint name="${robot_name}_joint_claw1_claw2" type="revolute">
-            <parent link="${robot_name}_link_claw1"/>
+            <parent link="${robot_name}_link_motor7"/>
             <child link="${robot_name}_link_claw2"/>
-            <origin xyz="0.03 0 0" rpy="0 0 0"/>
+            <origin xyz="0.03 0.0205 0" rpy="${-pi/2} 0 0"/>
             <axis xyz="0 0 1"/>
             <limit lower="${-170 * pi / 180}" upper="${170 * pi / 180}"
@@ -527,46 +561,4 @@
             mimic_joint="${robot_name}_joint_claw1_claw2"
             has_pid="false" multiplier="-1.0" max_effort="${max_effort}" />
-        <!-- joint between link_claw1 and link_claw1_end-->
-        <joint name="${robot_name}_joint_claw1_claw1_end" type="revolute">
-            <parent link="${robot_name}_link_claw1"/>
-            <child link="${robot_name}_link_claw1_end"/>
-            <origin xyz="-0.03858 -0.03487 0" rpy="0 0 0"/>
-            <axis xyz="0 0 1"/>
-            <limit lower="${-170 * pi / 180}" upper="${170 * pi / 180}"
-                effort="${max_effort}" velocity="${max_velocity}" />
-            <safety_controller soft_lower_limit="${-168 * pi / 180}"
-                     soft_upper_limit="${168 * pi / 180}"
-                     k_position="${safety_controller_k_pos}"
-                     k_velocity="${safety_controller_k_vel}"/>
-            <dynamics damping="${joint_damping}"/>
-            <mimic joint="${robot_name}_joint_7" multiplier="1.0" offset = "0"/>
-        </joint>
-        <xacro:mimic_joint_plugin_gazebo name_prefix="${robot_name}_joint_claw1_claw1_end"
-            parent_joint="${robot_name}_joint_7"
-            mimic_joint="${robot_name}_joint_claw1_claw1_end"
-            has_pid="false" multiplier="-1.0" max_effort="${max_effort}" />
-        <!-- link_claw1_end -->
-        <link name="${robot_name}_link_claw1_end">
-            <inertial>
-                <origin xyz="0.01175 -0.0276 -0.005" rpy="${pi/2} 0 1.903"/>
-                <mass value="0.006"/>
-                <inertia ixx="${scaling*0.0000001}" ixy="0" ixz="0" iyy="${scaling*0.000003}" iyz="0" izz="${scaling*0.000003}"/>
-            </inertial>
-            <visual>
-                <origin xyz="0.01175 -0.0276 -0.005" rpy="${pi/2} 0 1.903"/>
-                <geometry>
-                    <mesh filename="package://bbot_description/meshes/gripper_link3.stl" scale="1 1 1"/>
-                </geometry>
-                <material name="Orange"/>
-            </visual>
-            <collision>
-                <origin xyz="0.01175 -0.0276 -0.005" rpy="${pi/2} 0 1.903"/>
-                <geometry>
-                    <mesh filename="package://bbot_description/meshes/gripper_link3.stl" scale="1 1 1"/>
-                </geometry>
-                <material name="Orange"/>
-            </collision>
-        </link>
-        <!-- link_claw2 -->
         <link name="${robot_name}_link_claw2">
             <inertial>
@@ -590,9 +582,8 @@
             </collision>
         </link>
-        <!-- joint between link_claw2 and link_claw2_2-->
         <joint name="${robot_name}_joint_claw2_claw2_2" type="revolute">
-            <parent link="${robot_name}_link_claw2"/>
+            <parent link="${robot_name}_link_motor7"/>
             <child link="${robot_name}_link_claw2_2"/>
-            <origin xyz="-0.008 -0.024 0" rpy="0 0 0"/>
+            <origin xyz="0.022 .0205 0.024" rpy="${-pi/2} 0 0"/>
             <axis xyz="0 0 1"/>
             <limit lower="${-170 * pi / 180}" upper="${170 * pi / 180}"
@@ -609,5 +600,4 @@
             mimic_joint="${robot_name}_joint_claw2_claw2_2"
             has_pid="false" multiplier="-1.0" max_effort="${max_effort}" />
-        <!-- link_claw2_2 -->
         <link name="${robot_name}_link_claw2_2">
             <inertial>
@@ -631,5 +621,4 @@
             </collision>
         </link>
-        <!-- joint between link_claw2 and link_claw2_end-->
         <joint name="${robot_name}_joint_claw2_claw2_end" type="revolute">
             <parent link="${robot_name}_link_claw2"/>
@@ -650,5 +639,4 @@
             mimic_joint="${robot_name}_joint_claw2_claw2_end"
             has_pid="false" multiplier="1.0" max_effort="${max_effort}" />
-        <!-- link_claw2_end -->
         <link name="${robot_name}_link_claw2_end">
             <inertial>
@@ -674,5 +662,4 @@
         <xacro:bbot_gazebo robot_name="${robot_name}"/>
         <xacro:bbot_transmission hardware_interface="${hardware_interface}"/>
-        <!-- Aruco marker joints and links -->
         <joint name="${robot_name}_joint_baseplate_arucobase" type="fixed">
             <parent link="${robot_name}_link_baseplate"/>

Commit message: Updated joint limits to avoid self-collisions

File: bbot_description/urdf/bbot.xacro (robot description, xacro)
@@ -132,8 +132,8 @@
             <origin xyz="0 0 0" rpy="0 0 0"/>
             <axis xyz="0 0 1"/>
-            <limit lower="${-170 * pi / 180}" upper="${170 * pi / 180}"
-                effort="${max_effort}" velocity="${max_velocity}" />
-            <safety_controller soft_lower_limit="${-168 * pi / 180}"
-                     soft_upper_limit="${168 * pi / 180}"
+            <limit lower="${-95 * pi / 180}" upper="${95 * pi / 180}"
+                effort="${max_effort}" velocity="${max_velocity}" />
+            <safety_controller soft_lower_limit="${-93 * pi / 180}"
+                     soft_upper_limit="${93 * pi / 180}"
                      k_position="${safety_controller_k_pos}"
                      k_velocity="${safety_controller_k_vel}"/>
@@ -166,8 +166,8 @@
             <origin xyz="0.105 0 0" rpy="0 0 0"/>
             <axis xyz="0 0 1"/>
-            <limit lower="${-170 * pi / 180}" upper="${170 * pi / 180}"
-                effort="${max_effort}" velocity="${max_velocity}" />
-            <safety_controller soft_lower_limit="${-168 * pi / 180}"
-                     soft_upper_limit="${168 * pi / 180}"
+            <limit lower="${-100 * pi / 180}" upper="${100 * pi / 180}"
+                effort="${max_effort}" velocity="${max_velocity}" />
+            <safety_controller soft_lower_limit="${-95 * pi / 180}"
+                     soft_upper_limit="${95 * pi / 180}"
                      k_position="${safety_controller_k_pos}"
                      k_velocity="${safety_controller_k_vel}"/>
@@ -252,8 +252,8 @@
             <origin xyz="0 0 0" rpy="0 0 0"/>
             <axis xyz="0 0 1"/>
-            <limit lower="${-170 * pi / 180}" upper="${170 * pi / 180}"
-                effort="${max_effort}" velocity="${max_velocity}" />
-            <safety_controller soft_lower_limit="${-168 * pi / 180}"
-                     soft_upper_limit="${168 * pi / 180}"
+            <limit lower="${-120 * pi / 180}" upper="${120 * pi / 180}"
+                effort="${max_effort}" velocity="${max_velocity}" />
+            <safety_controller soft_lower_limit="${-118 * pi / 180}"
+                     soft_upper_limit="${118 * pi / 180}"
                      k_position="${safety_controller_k_pos}"
                      k_velocity="${safety_controller_k_vel}"/>
@@ -286,8 +286,8 @@
             <origin xyz="0 0 0.0625" rpy="${pi/2.0} ${-pi/2.0} 0"/>
             <axis xyz="0 0 1"/>
-            <limit lower="${-170 * pi / 180}" upper="${170 * pi / 180}"
-                effort="${max_effort}" velocity="${max_velocity}" />
-            <safety_controller soft_lower_limit="${-168 * pi / 180}"
-                     soft_upper_limit="${168 * pi / 180}"
+            <limit lower="${-30 * pi / 180}" upper="${120 * pi / 180}"
+                effort="${max_effort}" velocity="${max_velocity}" />
+            <safety_controller soft_lower_limit="${-28 * pi / 180}"
+                     soft_upper_limit="${118* pi / 180}"
                      k_position="${safety_controller_k_pos}"
                      k_velocity="${safety_controller_k_vel}"/>
@@ -346,8 +346,8 @@
             <origin xyz="0 -0.0332 0" rpy="${pi/2.0} 0 0"/>
             <axis xyz="0 0 1"/>
-            <limit lower="${-170 * pi / 180}" upper="${170 * pi / 180}"
-                effort="${max_effort}" velocity="${max_velocity}" />
-            <safety_controller soft_lower_limit="${-168 * pi / 180}"
-                     soft_upper_limit="${168 * pi / 180}"
+            <limit lower="${-120 * pi / 180}" upper="${120 * pi / 180}"
+                effort="${max_effort}" velocity="${max_velocity}" />
+            <safety_controller soft_lower_limit="${-118 * pi / 180}"
+                     soft_upper_limit="${118 * pi / 180}"
                      k_position="${safety_controller_k_pos}"
                      k_velocity="${safety_controller_k_vel}"/>
@@ -436,8 +436,8 @@
             <origin xyz="0 0 0" rpy="${-pi/2} 0 0"/>
             <axis xyz="0 0 1"/>
-            <limit lower="${-170 * pi / 180}" upper="${170 * pi / 180}"
-                effort="${max_effort}" velocity="${max_velocity}" />
-            <safety_controller soft_lower_limit="${-168 * pi / 180}"
-                     soft_upper_limit="${168 * pi / 180}"
+            <limit lower="${-175 * pi / 180}" upper="${175 * pi / 180}"
+                effort="${max_effort}" velocity="${max_velocity}" />
+            <safety_controller soft_lower_limit="${-170 * pi / 180}"
+                     soft_upper_limit="${170 * pi / 180}"
                      k_position="${safety_controller_k_pos}"
                      k_velocity="${safety_controller_k_vel}"/>

Commit message: Cut off wrist and updated testnode for testing each joint PD gains

File: bbot_description/urdf/bbot.xacro (robot description, xacro)
@@ -404,11 +404,11 @@
         </link>
         <!-- joint between gripper_palm and motor7 -->
-        <joint name="${robot_name}_joint_gripper_palm_motor7" type="fixed">
+        <!-- <joint name="${robot_name}_joint_gripper_palm_motor7" type="fixed">
             <parent link="${robot_name}_gripper_palm"/>
             <child link="${robot_name}_link_motor7"/>
             <origin xyz="-0.0155 -0.018 0.0513" rpy="0 0 0"/>
-        </joint>
+        </joint> -->
         <!-- motor 7 -->
-        <link name="${robot_name}_link_motor7">
+        <!-- <link name="${robot_name}_link_motor7">
             <inertial>
                 <origin xyz="0 0 0" rpy="${pi/2} 0 ${pi}"/>
@@ -659,5 +659,5 @@
                 <material name="Orange"/>
             </collision>
-        </link>
+        </link> -->
         <xacro:bbot_gazebo robot_name="${robot_name}"/>
         <xacro:bbot_transmission hardware_interface="${hardware_interface}"/>
